File: Gateway-RFM-RS485/V10/MySens-GWeasyRS485-Nano-V10-004.sch (EAGLE design)
At the start: 24 parts, among them IC1 ATSHA204A, IC2 REG1117, M1 ARDUINO-PRO-MINI-3.3V#NP

Commit message: Updates for GW + Mini
Parts:
- removed A4: (no value), pinhead:PINHD-1X1
- removed BH1750, I2C-1, I2C-2, MOTION: (no value), pinhead-2:PINHD-1X04_2.54-S
- removed HM1, HM3: (no value), SparkFun-Connectors:CONN_04
- removed HM2: (no value), SparkFun-Connectors:CONN_06SILK_FEMALE_PTH
- removed IC2: REG1117, burr-brown:REG1117
- removed L1: 4,7uH, SparkFun-Passives:INDUCTOR0805
- removed M1: ARDUINO-PRO-MINI-3.3V#NP, diy-modules:ARDUINO-PRO-MINI-3.3V#NP
- removed NMODULE: CONNECTOR_10DUPONT, TD-MySensors:CONNECTOR_10DUPONT
- removed R7: 10K, rcl:R-EU_R0805
- removed RAW: (no value), jumper:SJ
- removed STEPUP: TLV61224, TLV61224:TI-TLV61224
- added BOOST: R-78C1.8-1.0, dc-dc-converter:R-78C1.8-1.0
- added C3: 22p, rcl:C-EUC0805
- added C4: 0,1uF, rcl:C-EUC1206
- added F1: 1812L, ptc-littlefuse:1812L
- added JP1, JP10, JP11, JP12, JP13, JP14, JP15, JP16, JP3, JP6: (no value), pinhead-2:PINHD-1X04_2.54-S
- added MAX487: MAX481CPA, maxim-4:MAX481CPA
- added MYSX: (no value), pinhead-2:PINHD-2X08_2.54
- added R1: 1M, rcl:R-EU_R0805
- added R10, R9: 330R, rcl:R-EU_R0805
- added R2: 470K, rcl:R-EU_R0805
- added R6: 150R, rcl:R-EU_R0805
- added RAW(MYSX): (no value), jumper:SJ
- added REG1: LP2950Z, linear:LP2950Z
- added REG2: STEP-DWN-MP2307, diy-modules:DC-DC-STEP-DOWN-MP2307
- added REGULATED: (no value), con-wago-500:W237-103
- added RS1: MAX487ECSA+, Maxim_By_element14_Batch_1:MAX487ECSA+
- added U$2: NANO, Arduino-clone:NANO
- added U$3: 2.1MMJACKTHM, adafruit:2.1MMJACKTHM
- added X7: 1751264, con-phoenix-350:1751264
- C5: value 10uF -> (0.1uF); device SparkFun-Passives:CAP0805 -> rcl:C-EUC1206
- R3: value 10K -> (none)
Connections:
- removed net A2: HM2.1, M1.A2, NMODULE.2
- removed net A3: HM2.2, M1.A3, NMODULE.3
- removed net A6: M1.A6
- removed net A7: M1.A7
- removed net ATSHA_D7: HM3.4, IC1.SDA, M1.D7
- removed net N$13: L1.2, STEPUP.SW
- removed net RAW: M1.RAW, RAW.1
- removed net UREG: HM1.1, RAW.2
- new net 3.3V: MYSX.2
- new net 3V3: IC1.VCC, RFM69W.VCC, U$2.3.3V
- new net A: MAX487G$1.A, R6.1, R9.2, RS1.A, X7-2.K
- new net B: MAX487G$1.B, R10.1, R6.2, RS1.B, X7-3.K
- new net D7: IC1.SDA, U$2.D7
- new net N$20: U$2.AREF
- new net N$24: U$2.A2
- new net N$25: U$2.A3
- new net N$26: U$2.A4
- new net N$27: U$2.A5
- new net N$28: U$2.A6
- new net N$29: U$2.A7
- new net N$31: U$2.RST
- new net OUT: BOOST.VOUT, C1.1, C5.2, REG1.O, REG2.OUT+, REGULATED-1.KL
- new net RW: MYSX.1, RAW(MYSX).2, U$2.RAW
- new net VIN: F1.2, REGULATED-3.KL, U$3.TIP
- net A0: now also C4.2, MYSX.15, R1.2, R2.2, U$2.A0; no longer HM1.3, M1.A0
- net A1: now also MYSX.16, U$2.A1; no longer HM1.4, M1.A1, NMODULE.1
- net A4: now also JP10.4, JP6.4, MYSX.14; no longer A4.1, BH1750.3, HM2.3, I2C-1.3, I2C-2.3, M1.A4, NMODULE.6, R3.2
- net A5: now also JP10.3, JP6.3, MYSX.13; no longer BH1750.4, HM2.4, I2C-1.4, I2C-2.4, M1.A5, M1.GND.3, MOTION.4, NMODULE.7, R7.2
- net CSN: now also U$2.D10; no longer M1.D10
- net D3: now also MYSX.9, R3.2, U$2.D3; no longer HM2.5, M1.D3, NMODULE.4
- net D4: now also U$2.D4; no longer M1.D4, MOTION.3
- net D5: now also MYSX.11, U$2.D5; no longer M1.D5
- net D6: now also MYSX.12, U$2.D6; no longer HM2.6, M1.D6
- net D8: now also MAX487G$1.RO, RS1.RO, U$2.D8; no longer M1.D8
- net D9: now also MAX487G$1.DI, RS1.DI, U$2.D9; no longer HM3.3, M1.D9
- net GND: now also BOOST.GND, C3.1, C4.1, C5.1, JP1.1, JP1.2, JP1.3, JP1.4, JP10.2, JP6.2, MYSX.4, MYSX.8, R10.2, R2.1, REG1.GND, REG2.IN-, REG2.OUT-, REGULATED-2.KL, RS1.GND, U$2.GND, U$2.GND2, U$3.RING, X7-4.K; no longer BH1750.2, C5.2, HM1.2, HM3.1, I2C-1.2, I2C-2.2, IC2.GND, M1.GND.1, M1.GND.2, MOTION.2, NMODULE.9, STEPUP.GND
- net IN: now also BOOST.VIN, F1.1, R1.1, RAW(MYSX).1, REG1.I, REG2.IN+, X7-1.K; no longer C5.1, IC2.VIN, JP19.2, L1.1, NMODULE.10, STEPUP.EN, STEPUP.VBAT
- net IRQ: now also MAX487G$1.DE, MAX487G$1.RE/, MYSX.10, RS1.DE, RS1.~RE, U$2.D2; no longer M1.D2, NMODULE.5
- net MISO: now also U$2.D12; no longer M1.D12
- net MOSI: now also U$2.D11; no longer M1.D11
- net RESET: now also MYSX.7, U$2.RST1; no longer M1.RST.2
- net RX: now also MYSX.6, U$2.RX1; no longer M1.D0/RX
- net SCK: now also U$2.D13; no longer M1.D13
- net TX: now also MYSX.5, U$2.TX0; no longer M1.D1/TX
- net VCC: now also C3.2, JP10.1, JP19.2, JP3.1, JP3.2, JP3.3, JP3.4, JP6.1, MYSX.3, R9.1, RS1.VCC, U$2.5.5V; no longer BH1750.1, C1.1, HM3.2, I2C-1.1, I2C-2.1, IC1.VCC, IC2.VOUT, M1.VCC, MOTION.1, NMODULE.8, R7.1, RFM69W.VCC, STEPUP.FB, STEPUP.VOUT
Other:
- note added: "Connectors"
- note added: "Easy PCB - Rev 9"
- note added: "GND"
- note added: "MysX Connector"
- note added: "Power Converters"
- note added: "RAW"
- note added: "REGULATED"
- note added: "RS485"
- note added: "RS485 alternativ"
- note added: "Radio"
- note added: "Terminierung mit Pull-Widerständen. Zwischen A und B 150 Ohm, von A 330 Ohm nach VCC, von B 330 Ohm nach GND. Damit wird er Bus auf HIGH gehalten wenn Teilnehmer passiv sind. AC-Widerstand ca. bei 120 Ohm (150 // (330+330)) = 122,2."
- note added: "VDD-Config siehe 1Wire..."
- note removed: "??? B1 ??"
- note removed: "A3 für SHA Chip!"
- note removed: "Achtung nur wenn physikalisch an der Position von GND.3 der A5 Pin ist verbinden !!!"
- note removed: "Arduino Pro Mini"
- note removed: "BMP280"
- note removed: "Div"
- note removed: "Ereiterungen zur HM-Universalplatine kommen auf die Rückseite der Platine"
- note removed: "HomeMatic Universal (Pa-Pa)"
- note removed: "I2C Pullup"
- note removed: "Motion"
- note removed: "Neu in V1.0 -Pullups for IC2 possible -3V3 connected to VCC -Beschriftung "I2C" gefixt -Stepup integrated"
- note removed: "Radios (nur eins erlaubt!)"
- note removed: "Schraub 3,5mm"
- note removed: "easy MySensors-HM"
- moved on the sheet: ANT1, C1, C2, C5, IC1, JP19, R3, X2
