File: Gateway-RFM-RS485/V11/MySens-GWeasyRS485-Nano-V11-008.brd (EAGLE design)
At the start: 74 x 34 mm, 38 parts, among them IC1 ATSHA204A, X7 1751264

Commit message: Updates for GW + Mini
Parts:
- removed C10: 22p, rcl:C0805
- removed C9: 220p, rcl:C0805
- removed R4, R5: 60, rcl:R0805
- removed RS485: MAX487ECSA+, Maxim_By_element14_Batch_1:SOIC127P600X175-8N
- added C3: 22p, rcl:C0805
- added R10, R9: 330R, rcl:R0805
- added R6: 150R, rcl:R0805
- added RS1: MAX487ECSA+, Maxim_By_element14_Batch_1:SOIC127P600X175-8N
- moved R3 0.63 mm to (47.6, 10.8)
Connections:
- removed net N$21: C9.1, R4.1, R5.1
- net 3.3V: no longer IC1.2
- net 3V3: now also IC1.2
- net A: now also R6.1, R9.2, RS1.6; no longer R5.2, RS485.6
- net B: now also R10.1, R6.2, RS1.7; no longer R4.2, RS485.7
- net D8: now also RS1.1; no longer RS485.1
- net D9: now also RS1.4; no longer RS485.4
- net GND: now also C3.1, R10.2, RS1.5; no longer C10.1, C9.2, RS485.5
- net IRQ: now also RS1.2, RS1.3; no longer RS485.2, RS485.3
- net VCC: now also C3.2, R9.1, RS1.8; no longer C10.2, RS485.8
Routing:
- net D5: track 39.6 -> 72.2 mm, vias 1 -> 2
- net 3V3: track 47.2 -> 77.4 mm
- net D8: track 12.8 -> 35.0 mm
- net A4: track 74.8 -> 53.5 mm, vias 2 -> 1
- net D3: track 37.8 -> 56.9 mm, vias 2 -> 0
- net A: track 71.4 -> 54.7 mm, vias 0 -> 1
- net A0: track 68.2 -> 84.8 mm, vias 2 -> 3
- net N$21: track 16.2 -> 0.00 mm, vias 2 -> 0
- net GND: track 270.7 -> 256.6 mm, vias 2 -> 20
- net VCC: track 132.5 -> 145.7 mm
- net OUT: track 99.8 -> 87.6 mm, vias 3 -> 1
- net SCK: track 69.1 -> 80.7 mm
- net D6: track 53.5 -> 42.2 mm, vias 2 -> 0
- net B: track 40.7 -> 51.2 mm, vias 0 -> 2
- net A5: track 64.5 -> 54.8 mm, vias 2 -> 1
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Other:
- board text added: "-"
- board text added: "A4 SDA"
- board text added: "A5"
- board text added: "Fuse1"
- board text added: "IN"
- board text added: "Max487"
- board text added: "Mini360"
- board text added: "NanoGW 1.0a RS485, RFM69"
- board text added: "NanoGW 1.1 RS485, RFM69"
- board text added: "Proto typing"
- board text added: "VIN"
- board text removed: "MySensGW 0.2"
- board text removed: "NanoGW 1.0 RS485, RFM69"
