File: MySensors-HM-easy-PCB-RFM-CC1101-RS485-NRF/2_Mini/V01/MinieasyMySens-v01.sch (EAGLE design)
At the start: 38 parts, among them IC1 ATSHA204A, X7 1751264

Commit message: Updates for GW + Mini
Parts:
- removed BOOST: R-78C1.8-1.0, dc-dc-converter:R-78C1.8-1.0
- removed C10: 22p, rcl:C-EUC0805
- removed C4: 0,1uF, rcl:C-EUC1206
- removed C9: 220p, rcl:C-EUC0805
- removed F1: 1812L, ptc-littlefuse:1812L
- removed JP1, JP10, JP11, JP12, JP13, JP14, JP15, JP16, JP3, JP6: (no value), pinhead-2:PINHD-1X04_2.54-S
- removed MAX487: MAX481CPA, maxim-4:MAX481CPA
- removed MYSX: (no value), pinhead-2:PINHD-2X08_2.54
- removed R1: 1M, rcl:R-EU_R0805
- removed R2: 470K, rcl:R-EU_R0805
- removed R4, R5: 60, rcl:R-EU_R0805
- removed RAW(MYSX): (no value), jumper:SJ
- removed REG1: LP2950Z, linear:LP2950Z
- removed REG2: STEP-DWN-MP2307, diy-modules:DC-DC-STEP-DOWN-MP2307
- removed REGULATED: (no value), con-wago-500:W237-103
- removed RS485: MAX487ECSA+, Maxim_By_element14_Batch_1:MAX487ECSA+
- removed U$2: NANO, Arduino-clone:NANO
- removed U$3: 2.1MMJACKTHM, adafruit:2.1MMJACKTHM
- removed X7: 1751264, con-phoenix-350:1751264
- added A4: (no value), pinhead:PINHD-1X1
- added BH1750, I2C-1, I2C-2, MOTION: (no value), pinhead-2:PINHD-1X04_2.54-S
- added HM1, HM3: (no value), SparkFun-Connectors:CONN_04
- added HM2: (no value), SparkFun-Connectors:CONN_06SILK_FEMALE_PTH
- added IC2: REG1117, burr-brown:REG1117
- added L1: 4,7uH, SparkFun-Passives:INDUCTOR0805
- added M1: ARDUINO-PRO-MINI-3.3V#NP, diy-modules:ARDUINO-PRO-MINI-3.3V#NP
- added NMODULE: CONNECTOR_10DUPONT, TD-MySensors:CONNECTOR_10DUPONT
- added R7: 10K, rcl:R-EU_R0805
- added RAW: (no value), jumper:SJ
- added STEPUP: TLV61224, TLV61224:TI-TLV61224
- C5: value (0.1uF) -> 10uF; device rcl:C-EUC1206 -> SparkFun-Passives:CAP0805
- R3: value (none) -> 10K
Connections:
- removed net 3.3V: IC1.VCC, MYSX.2
- removed net 3V3: RFM69W.VCC, U$2.3.3V
- removed net A: MAX487G$1.A, R5.2, RS485.A, X7-2.K
- removed net B: MAX487G$1.B, R4.2, RS485.B, X7-3.K
- removed net D7: IC1.SDA, U$2.D7
- removed net N$20: U$2.AREF
- removed net N$21: C9.1, R4.1, R5.1
- removed net N$24: U$2.A2
- removed net N$25: U$2.A3
- removed net N$26: U$2.A4
- removed net N$27: U$2.A5
- removed net N$28: U$2.A6
- removed net N$29: U$2.A7
- removed net N$31: U$2.RST
- removed net OUT: BOOST.VOUT, C1.1, C5.2, REG1.O, REG2.OUT+, REGULATED-1.KL
- removed net RW: MYSX.1, RAW(MYSX).2, U$2.RAW
- removed net VIN: F1.2, REGULATED-3.KL, U$3.TIP
- new net A2: HM2.1, M1.A2, NMODULE.2
- new net A3: HM2.2, M1.A3, NMODULE.3
- new net A6: M1.A6
- new net A7: M1.A7
- new net ATSHA_D7: HM3.4, IC1.SDA, M1.D7
- new net N$13: L1.2, STEPUP.SW
- new net RAW: M1.RAW, RAW.1
- new net UREG: HM1.1, RAW.2
- net A0: now also HM1.3, M1.A0; no longer C4.2, MYSX.15, R1.2, R2.2, U$2.A0
- net A1: now also HM1.4, M1.A1, NMODULE.1; no longer MYSX.16, U$2.A1
- net A4: now also A4.1, BH1750.3, HM2.3, I2C-1.3, I2C-2.3, M1.A4, NMODULE.6, R3.2; no longer JP10.4, JP6.4, MYSX.14
- net A5: now also BH1750.4, HM2.4, I2C-1.4, I2C-2.4, M1.A5, M1.GND.3, MOTION.4, NMODULE.7, R7.2; no longer JP10.3, JP6.3, MYSX.13
- net CSN: now also M1.D10; no longer U$2.D10
- net D3: now also HM2.5, M1.D3, NMODULE.4; no longer MYSX.9, R3.2, U$2.D3
- net D4: now also M1.D4, MOTION.3; no longer U$2.D4
- net D5: now also M1.D5; no longer MYSX.11, U$2.D5
- net D6: now also HM2.6, M1.D6; no longer MYSX.12, U$2.D6
- net D8: now also M1.D8; no longer MAX487G$1.RO, RS485.RO, U$2.D8
- net D9: now also HM3.3, M1.D9; no longer MAX487G$1.DI, RS485.DI, U$2.D9
- net GND: now also BH1750.2, C5.2, HM1.2, HM3.1, I2C-1.2, I2C-2.2, IC2.GND, M1.GND.1, M1.GND.2, MOTION.2, NMODULE.9, STEPUP.GND; no longer BOOST.GND, C10.1, C4.1, C5.1, C9.2, JP1.1, JP1.2, JP1.3, JP1.4, JP10.2, JP6.2, MYSX.4, MYSX.8, R2.1, REG1.GND, REG2.IN-, REG2.OUT-, REGULATED-2.KL, RS485.GND, U$2.GND, U$2.GND2, U$3.RING, X7-4.K
- net IN: now also C5.1, IC2.VIN, JP19.2, L1.1, NMODULE.10, STEPUP.EN, STEPUP.VBAT; no longer BOOST.VIN, F1.1, R1.1, RAW(MYSX).1, REG1.I, REG2.IN+, X7-1.K
- net IRQ: now also M1.D2, NMODULE.5; no longer MAX487G$1.DE, MAX487G$1.RE/, MYSX.10, RS485.DE, RS485.~RE, U$2.D2
- net MISO: now also M1.D12; no longer U$2.D12
- net MOSI: now also M1.D11; no longer U$2.D11
- net RESET: now also M1.RST.2; no longer MYSX.7, U$2.RST1
- net RX: now also M1.D0/RX; no longer MYSX.6, U$2.RX1
- net SCK: now also M1.D13; no longer U$2.D13
- net TX: now also M1.D1/TX; no longer MYSX.5, U$2.TX0
- net VCC: now also BH1750.1, C1.1, HM3.2, I2C-1.1, I2C-2.1, IC1.VCC, IC2.VOUT, M1.VCC, MOTION.1, NMODULE.8, R7.1, RFM69W.VCC, STEPUP.FB, STEPUP.VOUT; no longer C10.2, JP10.1, JP19.2, JP3.1, JP3.2, JP3.3, JP3.4, JP6.1, MYSX.3, RS485.VCC, U$2.5.5V
Other:
- note added: "??? B1 ??"
- note added: "A3 für SHA Chip!"
- note added: "Achtung nur wenn physikalisch an der Position von GND.3 der A5 Pin ist verbinden !!!"
- note added: "Arduino Pro Mini"
- note added: "BMP280"
- note added: "Div"
- note added: "Ereiterungen zur HM-Universalplatine kommen auf die Rückseite der Platine"
- note added: "HomeMatic Universal (Pa-Pa)"
- note added: "I2C Pullup"
- note added: "Motion"
- note added: "Neu in V1.0 -Pullups for IC2 possible -3V3 connected to VCC -Beschriftung "I2C" gefixt -Stepup integrated V1.1 -Kurschluss VCC+GND durch Durchkontaktierung beim NModule-Pin3 beheben"
- note added: "Schraub 3,5mm"
- note added: "easy MySensors-HM"
- note removed: "Easy PCB - Rev 9"
- note removed: "GND"
- note removed: "MysX Connector"
- note removed: "Nrf24l01+ Radio"
- note removed: "Optional !"
- note removed: "Power Converters"
- note removed: "RAW"
- note removed: "REGULATED"
- note removed: "VDD-Config siehe 1Wire..."
- moved on the sheet: ANT1, C1, C2, C5, IC1, JP19, R3, X2
