File: MySensors-HM-easy-PCB-RFM-CC1101-RS485-NRF/2_Mini/V02/MinieasyMySens-V02-Build006.brd (EAGLE design)
At the start: 62 x 25 mm, 24 parts, among them IC1 ATSHA204A, IC2 REG1117, M1 ARDUINO-PRO-MINI-3.3V#NP

Commit message: Updates for GW + Mini
Parts:
- moved HM1 18.0 mm to (47.8, 21.7), flipped to the bottom, turned to 180 degrees
- moved HM2 18.0 mm to (58.0, 21.7), flipped to the bottom, turned to 270 degrees
- moved HM3 17.6 mm to (45.3, 3.90), flipped to the bottom, turned to 180 degrees
Connections:
- net A1: now also MOTION.4
- net A4: now also BH1750.4, I2C-1.4; no longer BH1750.3, I2C-1.3
- net A5: now also BH1750.3, I2C-1.3; no longer BH1750.4, I2C-1.4, MOTION.4
Routing:
- net A1: track 27.5 -> 67.7 mm, vias 0 -> 1
- net A2: track 25.2 -> 38.7 mm
- net VCC: track 129.1 -> 141.7 mm
- net SCK: track 33.2 -> 42.4 mm
- net ATSHA_D7: track 42.3 -> 34.0 mm, vias 1 -> 0
- net UREG: track 43.2 -> 35.1 mm, vias 0 -> 2
- net A4: track 87.5 -> 94.5 mm, vias 1 -> 2
- net D9: track 32.3 -> 25.7 mm
- net CSN: track 23.0 -> 28.6 mm
- net A3: track 25.1 -> 29.1 mm
- net IRQ: track 55.2 -> 51.6 mm, vias 0 -> 2
- net D4: track 35.4 -> 31.9 mm, vias 1 -> 2
- net IN: track 80.0 -> 76.6 mm
- net A0: track 20.8 -> 17.4 mm
- net MOSI: track 27.6 -> 30.4 mm
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Other:
- board size 62 x 25 mm -> 63 x 25 mm
- board text added: "A0"
- board text added: "A1"
- board text added: "A2"
- board text added: "A3"
- board text added: "A4"
- board text added: "A5"
- board text added: "D2"
- board text added: "D3"
- board text added: "D4"
- board text added: "D6"
- board text added: "GND"
- board text added: "IN"
- board text added: "SCL A5"
- board text added: "UREG"
- board text added: "easyMySens-Mini V0.2"
- board text removed: "easyMySens-Mini V0.1"
