File: MySensors-HM-easy-PCB-RFM-CC1101-RS485-NRF/2_Mini/V02/MinieasyMySens-V02-Build008.brd (EAGLE design)
At the start: 63 x 25 mm, 24 parts, among them IC1 ATSHA204A, IC2 REG1117, M1 ARDUINO-PRO-MINI-3.3V#NP

Commit message: Update RFM95
Parts:
- removed MOTION: (no value), pinhead-2:1X04-S
- added D4: (no value), pinhead:1X01
- added R4: 10k, rcl:M0805
- added U1: RFM69HCW, doug:RFM69HCW-XXXS2
- moved JP19 4.96 mm to (-1.27, 21.6), turned to 270 degrees
- moved ANT1 4.12 mm to (-1.94, 4.11), turned to 90 degrees
- moved X2 3.82 mm to (-4.19, 4.19)
Connections:
- removed net N$16: ANT1.1, RFM69W.ANT, X2.P
- new net ANT: ANT1.1, RFM69W.ANT, U1.ANT, X2.P
- new net N$1: U1.RESET
- new net N$14: U1.DIO2
- new net N$15: U1.DIO1
- net A1: no longer MOTION.4
- net CSN: now also R4.1, U1.NSS
- net D4: now also D4.1; no longer MOTION.3
- net GND: now also U1.GND_1, U1.GND_2, U1.GND_3; no longer MOTION.2
- net IRQ: now also U1.DIO0
- net MISO: now also U1.MISO
- net MOSI: now also U1.MOSI
- net SCK: now also U1.SCK
- net VCC: now also R4.2, U1.3.3V; no longer MOTION.1
Routing:
- net IRQ: track 51.6 -> 108.8 mm, vias 2 -> 1
- net GND: track 180.5 -> 236.8 mm, vias 13 -> 1
- net CSN: track 28.6 -> 54.6 mm, vias 0 -> 2
- net VCC: track 141.7 -> 167.1 mm, vias 4 -> 3
- net A1: track 67.7 -> 44.0 mm, vias 1 -> 0
- net ATSHA_D7: track 34.0 -> 50.3 mm
- net D4: track 31.9 -> 48.2 mm, vias 2 -> 0
- net IN: track 76.6 -> 88.4 mm
- net A5: track 79.3 -> 87.5 mm
- net RAW: track 50.4 -> 42.5 mm, vias 3 -> 0
- net ANT: track 0.00 -> 7.82 mm
- net N$16: track 4.17 -> 0.00 mm
- net MOSI: track 30.4 -> 26.5 mm
- net D6: track 30.0 -> 26.1 mm
- net A4: track 94.5 -> 98.0 mm, vias 2 -> 1
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Other:
- board size 63 x 25 mm -> 66.8 x 25 mm
