File: MySensors-HM-easy-PCB-RFM-CC1101-RS485-NRF/3_Nano/NanoMySens-v016.sch (EAGLE design)
At the start: 34 parts, among them IC1 ATSHA204A, IC31 ATMEGA168-TQFP, U1 RFM69HCW, Y2 8MHZ

Commit message: Update RFM95
Parts:
- added RFM69W: RFM69HW, hoperf:RFM69HW
Connections:
- net ANT: now also RFM69W.ANT
- net D10_SS: now also RFM69W.NSS
- net D11_MOSI: now also RFM69W.MOSI
- net D12_MISO: now also RFM69W.MISO
- net D13_SCK: now also RFM69W.SCK
- net D2_INT0: now also RFM69W.DIO0
- net GND: now also RFM69W.GNDA, RFM69W.GNDB
- net VCC: now also RFM69W.VCC
Other:
- note added: "Free Pins"
- note added: "Nur mit 3,3V Arduino!"
- note added: "RFM69(H)W"
Changed lines of the file:
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@@
 <?xml version="1.0" encoding="utf-8"?>
 <!DOCTYPE eagle SYSTEM "eagle.dtd">
-<eagle version="7.3.0">
+<eagle version="7.6.0">
 <drawing>
 <settings>
@@
 <part name="R1" library="rcl" deviceset="R-EU_" device="R0805" value="1M"/>
 <part name="R3" library="rcl" deviceset="R-EU_" device="R0805" value="470K"/>
+<part name="RFM69W" library="hoperf" deviceset="RFM69HW" device=""/>
+<part name="U$2" library="microbuilder" deviceset="GND" device=""/>
 </parts>
 <sheets>
@@
 <text x="165.1" y="-212.09" size="3.81" layer="95" ratio="15">HomeMatic Universal
 (Pa-Pa)</text>
+<text x="297.18" y="-81.28" size="1.778" layer="97">Free Pins</text>
+<text x="320.04" y="-33.02" size="1.778" layer="91">RFM69(H)W</text>
+<text x="314.96" y="-81.28" size="1.778" layer="97">Nur mit 3,3V Arduino!</text>
 </plain>
 <instances>
@@
 <instance part="R1" gate="G$1" x="271.78" y="-152.4"/>
 <instance part="R3" gate="G$1" x="289.56" y="-152.4"/>
+<instance part="RFM69W" gate="A" x="327.66" y="-43.18"/>
+<instance part="U$2" gate="G$1" x="350.52" y="-78.74"/>
 </instances>
 <busses>
@@
 <wire x1="294.64" y1="-152.4" x2="307.34" y2="-152.4" width="0.1524" layer="91"/>
 <label x="294.64" y="-152.4" size="1.778" layer="95"/>
+</segment>
+<segment>
+<pinref part="RFM69W" gate="A" pin="GNDB"/>
+<wire x1="345.44" y1="-73.66" x2="350.52" y2="-73.66" width="0.1524" layer="91"/>
+<pinref part="U$2" gate="G$1" pin="GND"/>
+<wire x1="350.52" y1="-73.66" x2="350.52" y2="-76.2" width="0.1524" layer="91"/>
+<pinref part="RFM69W" gate="A" pin="GNDA"/>
+<wire x1="345.44" y1="-63.5" x2="350.52" y2="-63.5" width="0.1524" layer="91"/>
+<wire x1="350.52" y1="-63.5" x2="350.52" y2="-73.66" width="0.1524" layer="91"/>
+<junction x="350.52" y="-73.66"/>
 </segment>
 </net>
@@
 <junction x="214.63" y="-151.13"/>
 </segment>
+<segment>
+<pinref part="RFM69W" gate="A" pin="VCC"/>
+<wire x1="307.34" y1="-73.66" x2="289.56" y2="-73.66" width="0.1524" layer="91"/>
+<label x="292.1" y="-73.66" size="1.778" layer="95"/>
+</segment>
 </net>
 <net name="TXD" class="0">
@@
 <wire x1="266.7" y1="-66.04" x2="246.38" y2="-66.04" width="0.1524" layer="91"/>
 <pinref part="U1" gate="G$1" pin="ANT"/>
+<label x="248.92" y="-66.04" size="1.778" layer="95"/>
+</segment>
+<segment>
+<pinref part="RFM69W" gate="A" pin="ANT"/>
+<wire x1="345.44" y1="-68.58" x2="355.6" y2="-68.58" width="0.1524" layer="91"/>
+<label x="347.98" y="-68.58" size="1.778" layer="95"/>
 </segment>
 </net>
@@
 <wire x1="102.87" y1="-240.03" x2="100.33" y2="-240.03" width="0.1524" layer="91"/>
 <label x="100.33" y="-240.03" size="1.27" layer="95" rot="R180" xref="yes"/>
+</segment>
+<segment>
+<pinref part="RFM69W" gate="A" pin="DIO0"/>
+<wire x1="307.34" y1="-43.18" x2="289.56" y2="-43.18" width="0.1524" layer="91"/>
+<label x="292.1" y="-43.18" size="1.778" layer="95"/>
 </segment>
 </net>
@@
 <pinref part="U1" gate="G$1" pin="NSS"/>
 </segment>
+<segment>
+<pinref part="RFM69W" gate="A" pin="NSS"/>
+<wire x1="345.44" y1="-43.18" x2="363.22" y2="-43.18" width="0.1524" layer="91"/>
+<label x="347.98" y="-43.18" size="1.778" layer="95"/>
+</segment>
 </net>
 <net name="D11_MOSI" class="0">
@@
 <label x="11.43" y="-255.27" size="1.778" layer="95"/>
 </segment>
+<segment>
+<pinref part="RFM69W" gate="A" pin="MOSI"/>
+<wire x1="345.44" y1="-48.26" x2="363.22" y2="-48.26" width="0.1524" layer="91"/>
+<label x="347.98" y="-48.26" size="1.778" layer="95"/>
+</segment>
 </net>
 <net name="D12_MISO" class="0">
@@
 <label x="11.43" y="-228.6" size="1.778" layer="95"/>
 </segment>
+<segment>
+<pinref part="RFM69W" gate="A" pin="MISO"/>
+<wire x1="345.44" y1="-53.34" x2="363.22" y2="-53.34" width="0.1524" layer="91"/>
+<label x="347.98" y="-53.34" size="1.778" layer="95"/>
+</segment>
 </net>
 <net name="D13_SCK" class="0">
@@
 <label x="11.43" y="-234.95" size="1.778" layer="95"/>
 </segment>
-</net>
+<segment>
+<pinref part="RFM69W" gate="A" pin="SCK"/>
+<wire x1="345.44" y1="-58.42" x2="363.22" y2="-58.42" width="0.1524" layer="91"/>
+<label x="347.98" y="-58.42" size="1.778" layer="95"/>
+</segment>
+</net>
