File: MySensors-HM-easy-PCB-RFM-CC1101-RS485-NRF/4_Nano-RS485/NanoRS485-MySens-v004.sch (EAGLE design)
At the start: 39 parts, among them IC1 ATSHA204A, IC31 ATMEGA168-TQFP, X1 1751280, Y2 8MHZ

Commit message: RS485 Nano with MySX2.6
Parts:
- removed C1: 10uF, SparkFun-Passives:CAP0805
- removed GND2, MISO, MOSI, NC, RST, RXD, SCK, TXD: WIREPADSMD1,27-254, wirepad:WIREPADSMD1,27-254
- removed HM1, HM3: (no value), SparkFun-Connectors:CONN_04
- removed HM2: (no value), SparkFun-Connectors:CONN_06SILK_FEMALE_PTH
- removed NMODULE: CONNECTOR_10DUPONT, TD-MySensors:CONNECTOR_10DUPONT
- removed STEPUP: TLV61224, TLV61224:TI-TLV61224
- removed X1: 1751280, con-phoenix-350:1751280
- added 3V3, A3, A4, A5, A6, D1, D10-SS, D11, D12, D13-SCK, D2, D3, D4, D5, D6, D7, D8, RES, VCC-LEGACY, VIN: WIREPADSMD1,27-254, wirepad:WIREPADSMD1,27-254
- added IC2: AT25DF512C-SSHN-B, microchip:25AA080SN
- added X2: 1751264, con-phoenix-350:1751264
- R2: value 10k -> 56k; device doug:RESISTOR0805-RES -> Discrete:R-0402
Connections:
- net N$24 renamed A7
- removed net ADC6: IC31.ADC6, R1.2, R3.1
- removed net CE-A: HM3.3, IC31.PB1(OC1A)
- removed net IRQ: RS485.DE, RS485.~RE
- removed net N$10: IC31.PD4(XCK/T0)
- removed net N$9: IC31.PD5(T1)
- removed net TXD: IC31.PD1(TXD), TXD.P
- new net 3V3: 3V3.P
- new net A6: A6.P, IC31.ADC6, R1.2, R3.1
- new net D1-TXD: D1.P, IC31.PD1(TXD)
- new net D4: D4.P, IC31.PD4(XCK/T0)
- new net D5: D5.P, IC31.PD5(T1)
- net A: no longer X1-3.K
- net A0: no longer HM1.3
- net A1: no longer HM1.4, NMODULE.1
- net A2: no longer HM2.1, NMODULE.2
- net A3: now also A3.P; no longer HM2.2, NMODULE.3
- net A4: now also A4.P; no longer HM2.3, NMODULE.6
- net A5: now also A5.P; no longer HM2.4, NMODULE.7
- net B: no longer X1-4.K
- net D10_SS: now also D10-SS.P; no longer R2.1
- net D11_MOSI: now also D11.P, IC2.SI; no longer MOSI.P
- net D12_MISO: now also D12.P, IC2.SO; no longer MISO.P
- net D13_SCK: now also D13-SCK.P, IC2.SCK; no longer SCK.P
- net D2_INT0: now also D2.P, RS485.DE, RS485.~RE; no longer NMODULE.5
- net D3: now also D3.P; no longer HM2.5, NMODULE.4
- net D6: now also D6.P; no longer HM2.6
- net D7-ATSHA: now also D7.P; no longer HM3.4
- net D8: now also D8.P, IC2.!CS, R2.1
- net D9: now also IC31.PB1(OC1A)
- net GND: now also IC2.GND; no longer C1.2, GND2.P, HM1.2, HM3.1, NMODULE.9, STEPUP.GND, X1-5.K
- net IN: no longer X1-1.K
- net N$13: no longer STEPUP.SW
- net RESET: now also RES.P; no longer RST.P
- net RXD: no longer RXD.P
- net UREG: no longer X1-2.K
- net VCC: now also IC2.!HOLD, IC2.!WP, IC2.VCC, VCC-LEGACY.P; no longer HM3.2, NMODULE.8, STEPUP.FB, STEPUP.VOUT, X1-6.K
- net VIN: now also VIN.P; no longer C1.1, HM1.1, NMODULE.10, STEPUP.EN, STEPUP.VBAT
Other:
- note added: "1 Vraw (typically unregulated voltage, either from motherboard to daughterboard or vice versa) Motherboard should have a jumper to cut onboard Vraw source if daughterboard provides Vraw. Be sure to check motherboard constraints on Vraw before connecting a daughterboard that provides Vraw (for over voltage protection). Should be able to source at least 100mA and all boards are recommended to suppo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"
- note added: "mySX V2.6"
- note removed: "A3 für SHA Chip!"
- note removed: "Connectors"
- note removed: "HomeMatic Universal (Pa-Pa)"
- note removed: "NModule Extensions"
- note removed: "Prog"
- note removed: "Transceiver"
- moved on the sheet: C10, C14, C15, C31, C32, IC31, R34, R4, R5, R6, R7, RS485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
