File: MySensors-HM-easy-PCB-RFM-CC1101-RS485-NRF/4_Nano-RS485/NanoRS485-MySens-v005.brd (EAGLE design)
At the start: 25 x 38.7 mm, 46 parts, among them IC1 ATSHA204A, IC2 AT25DF512C-SSHN-B, IC31 ATMEGA168-TQFP, X2 1751264, Y2 8MHZ

Commit message: 1117
Parts:
- added IC3: REG1117, burr-brown:SOT223
- moved C31 1.63 mm to (6.35, 31.8), turned to 180 degrees
- moved C5 1.27 mm to (19.1, 27.8)
- moved C32 0.25 mm to (12.7, 31.8)
- moved R34 0.25 mm to (17.8, 31.8)
Connections:
- removed net N$13: L1.2
- new net RAW: IC3.3, L1.2
- net GND: now also IC3.1
- net VCC: now also IC3.2
