File: MySensors-HM-easy-PCB-RFM-CC1101-RS485-NRF/4_Nano-RS485/NanoRS485-MySens-v005.sch (EAGLE design)
At the start: 46 parts, among them IC1 ATSHA204A, IC2 AT25DF512C-SSHN-B, IC31 ATMEGA168-TQFP, X2 1751264, Y2 8MHZ

Commit message: 1117
Parts:
- added IC3: REG1117, burr-brown:REG1117
Connections:
- removed net N$13: L1.2
- new net RAW: IC3.VIN, L1.2
- net GND: now also IC3.GND
- net VCC: now also IC3.VOUT
Other:
- note added: "Regulator"
- note removed: "Stepup"
- moved on the sheet: C5, L1, R1, R3
