File: MySensors-HM-easy-PCB-RFM-CC1101-RS485-NRF/4_Nano-RS485/NanoRS485-MySens-v010-both-connectors.sch (EAGLE design)
At the start: 47 parts, among them IC1 ATSHA204A, IC2 AT25DF512C-SSHN-B, IC3 REG1117, IC31 ATMEGA168-TQFP, X2 1751264, Y2 8MHZ

Commit message: RS485 New SubBoard
Parts:
- removed CONFIG: DTSM-3, mechanics:DTSM-3
- added JP1: JUMPER-SMT_2_NC_TRACE_SILK, SparkFun-Jumpers:JUMPER-SMT_2_NC_TRACE_SILK
- added SV1: (no value), con-lstb:MA10-2
- R2: device Discrete:R-0402 -> resistor:R-EU_M0805
Connections:
- removed net 3V3: 3V3.P
- new net VCC1: IC2.!HOLD, IC2.!WP, IC2.VCC, JP1.1, R2.2
- net A0: now also SV1.8, VCC-LEGACY.P
- net A3: now also SV1.15
- net A4: now also SV1.16
- net D1-TXD: now also SV1.5
- net D10_SS: now also SV1.20
- net D11_MOSI: now also SV1.17
- net D12_MISO: now also SV1.18
- net D13_SCK: now also SV1.19
- net D2_INT0: no longer D2.P
- net D3: now also SV1.9
- net D4: now also SV1.10
- net D5: now also SV1.11
- net D6: now also SV1.12
- net D7-ATSHA: now also SV1.13
- net D8: now also SV1.14; no longer CONFIG.2
- net GND: now also SV1.4; no longer CONFIG.1
- net RESET: now also SV1.7
- net RXD: now also D2.P, SV1.6
- net VCC: now also 3V3.P, JP1.2, SV1.2, SV1.3; no longer IC2.!HOLD, IC2.!WP, IC2.VCC, R2.2, VCC-LEGACY.P
- net VIN: now also SV1.1
Other:
- note removed: "Config"
