File: MySensors-HM-easy-PCB-RFM-CC1101-RS485-NRF/4_Nano-RS485/NanoRS485-MySens-v023.sch (EAGLE design)
At the start: 54 parts, among them IC1 ATSHA204A, IC2 AT25DF512C-SSHN-B, IC3 REG1117, IC31 ATMEGA168-TQFP, X2 1751264, Y2 8MHZ

Commit message: Nano RS485
Parts:
- removed JP11, JP12, JP17, JP22, JP4, JP9: (no value), pinhead-2:PINHD-1X04_2.54-S
- added SV2: (no value), con-lstb:MA10-2
Connections:
- net A0: now also SV2.8
- net A3: now also SV2.15
- net A4: now also SV2.16
- net D1-TXD: now also SV2.5
- net D10_SS: now also SV2.20
- net D11_MOSI: now also SV2.17
- net D12_MISO: now also SV2.18
- net D13_SCK: now also SV2.19
- net D3: now also SV2.9
- net D4: now also SV2.10
- net D5: now also SV2.11
- net D6: now also SV2.12
- net D7-ATSHA: now also SV2.13
- net D8: now also SV2.14
- net GND: now also SV2.4
- net RESET: now also SV2.7
- net RXD: now also SV2.6
- net VCC: now also SV2.2, SV2.3
- net VIN: now also SV2.1
Other:
- note added: "ExtensionPCB"
