File: GW-Sens-RS485-ProMicro/MySens-GWeasySensRS485-003.sch (EAGLE design)
At the start: 19 parts, among them IC1 ATSHA204A, X7 1751264

Commit message: RS485 Pro Mico ready for test
Parts:
- removed J4: (no value), con-amp:215878-2
- added MAX487: MAX481CPA, maxim-4:MAX481CPA
- added R1, R2: 10K, rcl:R-EU_R0805
- J1: device con-amp:215878-2 -> con-amp:557570-1
Connections:
- removed net A4: JP10.4
- removed net A5: JP10.3
- removed net D7: IC1.SDA
- removed net RW: RAW.2
- new net D2: JP10.4, R1.2
- new net D3: JP10.3, R2.2
- net 7: now also IC1.SDA
- net A: now also J1-1.1, J1-2.1, MAX487G$1.A; no longer J1.1, J4.1
- net B: now also J1-1.2, J1-2.2, MAX487G$1.B; no longer J1.2, J4.2
- net GND: now also J1-1.6, J1-1.8, J1-2.6, J1-2.8; no longer J1.6, J1.8, J4.6, J4.8
- net IN: now also J1-1.3, J1-1.7, J1-2.3, J1-2.7; no longer 1117.VIN, C5.1, J1.3, J1.7, J4.3, J4.7, RAW.1
- net IRQ: now also MAX487G$1.DE, MAX487G$1.RE/
- net N$1: now also J1-2.4; no longer J4.4
- net N$10: now also J1-1.5; no longer J1.5
- net N$5: now also J1-2.5; no longer J4.5
- net N$9: now also J1-1.4; no longer J1.4
- net RAW: now also 1117.VIN, C5.1, RAW.2
- net RX: now also MAX487G$1.RO
- net TX: now also MAX487G$1.DI
- net VCC: now also R1.1, R2.1, RAW.1
Other:
- note added: "RS485 alternativ"
- moved on the sheet: C1, IC1
