File: Experimental/GW-Maple-RS485-RFM/MySens-easyRS485-BluePill-V02-011.sch (EAGLE design)
At the start: 40 parts, among them IC1 ATSHA204A, U1 RFM69HCW, U2 RFM69HCW, X3 1751264

Commit message: BluePill, MiniRS485 Sensor+Gateway
Parts:
- removed 1117: REG1117, burr-brown:REG1117
- removed BOOST: R-78C1.8-1.0, dc-dc-converter:R-78C1.8-1.0
- removed C2: 10uF, rcl:CPOL-EUR/2012-12W
- removed C6: 22pF, rcl:C-EUC0805
- removed F1: 1812L, ptc-littlefuse:1812L
- removed J2: (no value), con-amp:557570-1
- removed JP1, JP10, JP11, JP12, JP15, JP2, JP3, JP4, JP5, JP6, JP7, JP8, JP9, UART2: (no value), pinhead-2:PINHD-1X04_2.54-S
- removed MAX487: MAX481CPA, maxim-4:MAX481CPA
- removed U$2: MAPLEMINI, maplemini-small:MAPLEMINI
- added BH1750, I2C-1, I2C-2, STEPDWN: (no value), pinhead-2:PINHD-1X04_2.54-S
- added C1: 0.1uF, rcl:C-EUC1206
- added C4: 10uF, rcl:C-EUC1210
- added C7: 22pF, rcl:C-EUC0805
- added F2: 1812L, ptc-littlefuse:1812L
- added IC2: LAN-USR-ES1, Martin-Communication:LAN-USR-ES1
- added IC5: LD117ADT50TR, v-reg:LD117ADT50TR
- added IC6: LM1117MPX-ADJ, lm1117:LM1117MPX-ADJ
- added J1: (no value), RJ45:RJ45_2X_NARROW_SHILDPINS_NOCASE
- added LAN1, LAN2: JUMPER-SMT_2_NC_PASTE_SILK, SparkFun-Jumpers:JUMPER-SMT_2_NC_PASTE_SILK
- added R2: 1M, rcl:R-EU_R0805
- added R3: 470K, rcl:R-EU_R0805
- added SV2: (no value), con-Pinheader:MA11-2
- added U$4: BLUEPILL, stm32duino boards:BLUEPILL
- added V2: (no value), pinhead:PINHD-1X1
- C5: value 0.1uF -> 10uF; device rcl:C-EUC1206 -> rcl:CPOL-EUR/2012-12W
- renumbered IC1 to CRYPTO
Connections:
- removed net +5V: U$2.VIN
- removed net B6_TX: MAX487G$1.DI, RS1.DI, U$2.16/PWM/I2C1_SCL
- removed net B7_RX: MAX487G$1.RO, RS1.RO, U$2.15/PWM/I2C1_SDA
- removed net CC_CS1: U$2.12
- removed net CC_CS3: U$2.3/PWM/AIN
- removed net CC_IN_1: U$2.18
- removed net CC_OUT_1: U$2.17
- removed net CC_OUT_2: U$2.13
- removed net IN: F1.1, J2-1.3, J2-1.7, J2-2.3, J2-2.7, X3-1.K
- removed net N$2: J2-1.4
- removed net N$3: J2-1.5
- removed net N$6: J2-2.4
- removed net N$7: J2-2.5
- removed net NRESET: U$2.RESET
- removed net OUT: BOOST.VOUT
- removed net RX-MAPLE: U$2.8/PWM/AIN/RX2, UART2.3
- removed net RX_DBG: DBG.3, U$2.25/PWM/RX1
- removed net SCL: JP10.3, JP2.3, JP5.3, U$2.1/TX3/I2C2_SCL
- removed net SDA: JP10.4, JP2.4, JP5.4, U$2.0/RX3/I2C2_SDA
- removed net SWCLK/TCK: U$2.21
- removed net SWDIO/TMS: U$2.22
- removed net SWO/TDO: U$2.19
- removed net TDI: U$2.20
- removed net TX-MAPLE: U$2.9/PWM/AIN/TX2, UART2.2
- removed net TX_DBG: DBG.2, U$2.26/PWM/TX1
- new net 4: J1-1.4, LAN1.1
- new net 5: J1-1.5, LAN2.1
- new net 5V: C4.1, IC2.V+, IC2.V+@1, IC5.OUT, IC6.OUT, IC6.OUT1, STEPDWN.1, STEPDWN.4, U$4.5V, V2.1
- new net A0: SV2.21
- new net A1: SV2.22
- new net A2: SV2.16
- new net A3: SV2.15
- new net A4: BH1750.4, I2C-1.4, I2C-2.3, SV2.14
- new net A5: BH1750.3, I2C-1.3, I2C-2.4, SV2.13
- new net A7: SV2.8
- new net CSN1: U$4.PA4/A4/SS1
- new net D10_SS: SV2.20
- new net D11_MOSI: SV2.17
- new net D12_MISO: SV2.18
- new net D13_SCK: SV2.19
- new net D2: SV2.9
- new net D3: SV2.10
- new net D5: SV2.11
- new net D6: SV2.12
- new net MISO1: U$4.PA6/A2/MISO1
- new net MOSI1: U$4.PA7/A1/M0SI1
- new net N$12: U$4.PC14
- new net N$13: U$4.PC15
- new net N$25: U$4.PB1
- new net N$33: IC2.!INT!
- new net N$35: U$4.PB9
- new net N$36: U$4.PB8
- new net N$39: U$4.PB5
- new net N$40: U$4.PB4
- new net N$41: U$4.PB3
- new net N$42: U$4.PA15
- new net N$43: U$4.PA12/USB+
- new net N$44: U$4.PA11/USB-
- new net PB0: R2.2, R3.2, U$4.PB0/A0
- new net RESET: SV2.7, U$4.RESET
- new net RX0: SV2.6
- new net RX1: DBG.2, U$4.PA10/RX1
- new net RX2: RS1.RO, U$4.PA3/A5/RX2
- new net SCK1: U$4.PA5/A3/SCK1
- new net SCL1: U$4.PB6/SCL1
- new net SCL2: U$4.PB10/TX3/SCL2
- new net SDA1: U$4.PB7/SDA1
- new net SDA2: U$4.PB11/RX3/SDA2
- new net TX1: DBG.3, SV2.5, U$4.PA9/TX1
- new net TX2: RS1.DI, U$4.PA2/A6/TX2
- new net UREG: C1.1, F2.1, IC5.IN, IC6.IN, R2.1, STEPDWN.3, SV2.1
- net A: now also J1-1.1, J1-2.1, LAN1.2; no longer J2-1.1, J2-2.1, MAX487G$1.A
- net B: now also J1-1.2, J1-2.2, LAN2.2; no longer J2-1.2, J2-2.2, MAX487G$1.B
- net CSN: no longer U$2.7/AIN/SPI1_SS
- net CSN2: now also IC2.!SCS!, U$4.PB12/SS2; no longer U$2.31/SPI2_SS
- net GND: now also BH1750.2, C1.2, C4.2, C5.-, C7.2, I2C-1.2, I2C-2.2, IC2.GND, IC2.GND@1, IC2.GND@2, IC5.ADJ, IC6.ADJ, J1-1.6, J1-1.8, J1-1.S1, J1-1.S2, J1-2.6, J1-2.8, R3.1, STEPDWN.2, SV2.4, U$4.GND/1, U$4.GND/2, U$4.GND/3; no longer 1117.GND, BOOST.GND, C2.-, C5.2, C6.2, J2-1.6, J2-1.8, J2-2.6, J2-2.8, JP1.1, JP1.2, JP1.3, JP1.4, JP10.2, JP2.2, JP5.2, U$2.2/BOOT1, U$2.AV-, U$2.GND, UART2.4
- net IRQ: now also U$4.PA0/A8; no longer MAX487G$1.DE, MAX487G$1.RE/, U$2.11/PWM/AIN
- net IRQ2: now also U$4.PA1/A7; no longer U$2.10/PWM/AIN
- net MISO: no longer U$2.5/PWM/AIN/SPI1_MISO
- net MISO2: now also IC2.MISO, U$4.PB14/MIS02; no longer U$2.29/SPI2_MISO
- net MOSI: no longer U$2.4/PWM/AIN/SPI1_MOSI
- net MOSI2: now also IC2.MOSI, U$4.PB15/MOSI2; no longer U$2.28/SPI2_MOSI
- net PC13: now also U$4.PC13; no longer U$2.14
- net SCK: no longer U$2.6/AIN/SPI1_SCK
- net SCK2: now also IC2.SCLK, U$4.PB13/SCK2; no longer U$2.30/SPI2_SCK
- net VCC: now also BH1750.1, C5.+, C7.1, I2C-1.1, I2C-2.1, SV2.2, SV2.3, U$4.3V3, U$4.3V3/1; no longer 1117.VOUT, C2.+, C6.1, JP10.1, JP2.1, JP3.1, JP3.2, JP3.3, JP3.4, JP5.1, U$2.AV+, U$2.VCC, UART2.1
- net VIN: now also F2.2, J1-1.3, J1-1.7, J1-2.3, J1-2.7, X3-1.K; no longer 1117.VIN, BOOST.VIN, C5.1, F1.2
- net WIZ_RST: now also IC2.RES, U$4.PA8; no longer U$2.27/PWM
Other:
- note added: "1 Vraw (typically unregulated voltage, either from motherboard to daughterboard or vice versa) Motherboard should have a jumper to cut onboard Vraw source if daughterboard provides Vraw. Be sure to check motherboard constraints on Vraw before connecting a daughterboard that provides Vraw (for over voltage protection). Should be able to source at least 100mA and all boards are recommended to suppo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"
- note added: "8 7 6 5 4 3 2 1 Pair 4 1 2 gn3 ws3"
- note added: "BMP280"
- note added: "Blue-Pill"
- note added: "Div"
- note added: "Neu in V1.0 -Pullups for IC2 possible -3V3 connected to VCC -Beschriftung "I2C" gefixt -Stepup integrated V1.1 -Kurschluss VCC+GND durch Durchkontaktierung beim NModule-Pin3 behoben -SDA /SCL getauscht V1.2 -kein NModul + PaPa Connector mehr -33mm Breite"
- note added: "Nicht nutzbar mit LAN Modul"
- note added: "RS485 Connectors"
- note added: "Regulator"
- note removed: "1 2 3 4 5 6 7 8 Pair 2 1 4 ws3 gn3"
- note removed: "MAPLE-Mini"
- note removed: "Nur mit 3,3V Arduino!"
- note removed: "RS485 alternativ"
- note removed: "siehe MySensors"
