File: Experimental/GW-STM32-RS485-RFM/MySens-easyRS485-BluePill-V03-not-ordered-015.sch (EAGLE design)
At the start: 37 parts, among them IC2 LAN-USR-ES1, IC5 LD117ADT50TR, IC6 LM1117MPX-ADJ, U1 RFM69HCW, U2 RFM69HCW, X3 1751264

Commit message: STM32 and other Updates
Parts:
- added C2: 22pF, rcl:C-EUC0805
- added CC0: CC1101, wireless:CC1101_MODULE1SMD
- added X5: (no value), adafruit:SMACONNECTOR_EDGE
- renumbered SV2 to MYSX
Connections:
- new net ANT0: CC0.ANT, X5.ANT
- net GND: now also C2.1, CC0.GND@1, CC0.GND@2, CC0.GND@3, X5.GND1, X5.GND2, X5.GND3, X5.GND4
- net PA0: now also CC0.GDO2
- net PA1: now also CC0.GDO0
- net PA4: now also CC0.CSN
- net PA5: now also CC0.SCLK
- net PA6: now also CC0.MISO
- net PA7: now also CC0.MOSI
- net VCC: now also C2.2, CC0.VCC
Other:
- note added: "CC1101"
- note added: "Radio 0"
