File: Experimental/GW-STM32-RS485-RFM/MySens-easyRS485-BluePill-MAPLE-V04-not-ordered-017.brd (EAGLE design)
At the start: 90 x 33 mm, 40 parts, among them IC2 LAN-USR-ES1, IC5 LD117ADT50TR, IC6 LM1117MPX-ADJ, U1 RFM69HCW, U2 RFM69HCW, X3 1751264

Commit message: stm32 update
Parts:
- added U$2: MAPLEMINI, maplemini-small:20-DIP
- moved C2 90.6 mm to (-6.99, 59.1)
- moved X5 75.6 mm to (29.2, 40.0), turned to 270 degrees
- moved CC0 51.2 mm to (36.2, 14.0), turned to 90 degrees
- moved RFM69W 39.6 mm to (43.8, 37.8), flipped to the top, turned to 180 degrees
- moved RFM69W1 36.3 mm to (46.4, 1.67), flipped to the bottom, turned to 0 degrees
- moved DBG 29.6 mm to (79.8, 47.6)
- moved IC2 27.5 mm to (58.4, 33.4), turned to 0 degrees
- moved IC6 22.9 mm to (51.8, 48.3)
- moved IC5 22.5 mm to (52.5, 48.3)
- moved BH1750 22.2 mm to (66.0, 50.2)
- moved RS1 17.8 mm to (44.7, -6.24)
- moved I2C-2 17.0 mm to (51.8, -12.1)
- moved R1 14.5 mm to (44.1, 41.9)
- moved C7 12.7 mm to (48.7, -1.27)
- moved MYSX 12.3 mm to (85.1, 36.8)
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Connections:
- new net +5V: U$2.21
- new net PA13: U$2.11
- new net PA14: U$2.10
- new net PB2: U$2.24
- new net RAW: U$2.38
- net GND: now also U$2.2, U$2.39
- net PA0: now also U$2.33
- net PA1: now also U$2.32
- net PA10: now also U$2.14
- net PA11: now also U$2.13
- net PA12: now also U$2.12
- net PA15: now also U$2.9
- net PA2: now also U$2.31
- net PA3: now also U$2.30
- net PA4: now also U$2.29
- net PA5: now also U$2.28
- net PA6: now also U$2.27
- net PA7: now also U$2.26
- net PA8: now also U$2.16
- net PA9: now also U$2.15
- net PB0: now also U$2.25
- net PB10: now also U$2.23
- net PB11: now also U$2.22
- net PB12: now also U$2.20
- net PB13: now also U$2.19
- net PB14: now also U$2.18
- net PB15: now also U$2.17
- net PB3: now also U$2.8
- net PB4: now also U$2.7
- net PB5: now also U$2.6
- net PB6: now also U$2.5
- net PB7: now also U$2.4
- net PB8: now also U$2.3
- net PC13: now also U$2.37
- net PC14: now also U$2.36
- net PC15: now also U$2.35
- net RESET: now also U$2.34
- net VCC: now also U$2.1, U$2.40
Routing:
- net VCC: track 179.9 -> 0.00 mm, vias 4 -> 0
- net PA0: track 162.5 -> 0.00 mm
- net UREG: track 135.8 -> 0.00 mm, vias 1 -> 0
- net 3V3: track 124.5 -> 0.00 mm, vias 3 -> 0
- net PB12: track 92.6 -> 0.00 mm, vias 3 -> 0
- net 5V: track 90.2 -> 0.00 mm, vias 1 -> 0
- net B: track 89.3 -> 0.00 mm
- net PA4: track 82.9 -> 0.00 mm, vias 2 -> 0
- net PA5: track 80.4 -> 0.00 mm, vias 3 -> 0
- net PB13: track 76.1 -> 0.00 mm, vias 2 -> 0
- net PA7: track 74.6 -> 0.00 mm, vias 1 -> 0
- net PB14: track 74.3 -> 0.00 mm, vias 1 -> 0
- net A: track 72.3 -> 0.00 mm, vias 2 -> 0
- net PA6: track 65.8 -> 0.00 mm, vias 1 -> 0
- net PB15: track 64.1 -> 0.00 mm, vias 4 -> 0
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- removed copper zone on layer 1, net GND
- removed copper zone on layer 16, net GND
Other:
- board size 90 x 33 mm -> 100 x 40 mm
