File: Experimental/GW-STM32-RS485-RFM/MySens-easyRS485-BluePill-MAPLE-V05-not-ordered-018.brd (EAGLE design)
At the start: 100 x 40 mm, 41 parts, among them IC2 LAN-USR-ES1, IC5 LD117ADT50TR, IC6 LM1117MPX-ADJ, U1 RFM69HCW, U2 RFM69HCW, X3 1751264

Commit message: CAN Sensor / Gateway
Connections:
- net PA0: no longer RFM69W.DIO0, U1.DIO0
- net PA2: now also MYSX.21, RFM69W.DIO0, U1.DIO0; no longer MYSX.15
- net PA3: now also MYSX.22; no longer MYSX.16
- net PA4: no longer CC0.CSN
- net PA5: no longer CC0.SCLK
- net PA6: no longer CC0.MISO
- net PA7: no longer CC0.MOSI
- net PB0: now also MYSX.15; no longer MYSX.21
- net PB1: now also MYSX.8; no longer MYSX.22
- net PB10: now also MYSX.13; no longer MYSX.8
- net PB11: now also MYSX.14
- net PB12: now also CC0.CSN
- net PB13: now also CC0.SCLK
- net PB14: now also CC0.MISO
- net PB15: now also CC0.MOSI
- net PB8: now also MYSX.16; no longer MYSX.13
- net PB9: no longer MYSX.14
