File: Experimental/GW-STM32-RS485-RFM/MySens-easyRS485-BluePill-MAPLE-V05-not-ordered-018.sch (EAGLE design)
At the start: 41 parts, among them IC2 LAN-USR-ES1, IC5 LD117ADT50TR, IC6 LM1117MPX-ADJ, U1 RFM69HCW, U2 RFM69HCW, X3 1751264

Commit message: CAN Sensor / Gateway
Connections:
- net PA0: no longer RFM69W.DIO0, U1.DIO0
- net PA2: now also MYSX.21, RFM69W.DIO0, U1.DIO0; no longer MYSX.15
- net PA3: now also MYSX.22; no longer MYSX.16
- net PA4: no longer CC0.CSN
- net PA5: no longer CC0.SCLK
- net PA6: no longer CC0.MISO
- net PA7: no longer CC0.MOSI
- net PB0: now also MYSX.15; no longer MYSX.21
- net PB1: now also MYSX.8; no longer MYSX.22
- net PB10: now also MYSX.13; no longer MYSX.8
- net PB11: now also MYSX.14
- net PB12: now also CC0.CSN
- net PB13: now also CC0.SCLK
- net PB14: now also CC0.MISO
- net PB15: now also CC0.MOSI
- net PB8: now also MYSX.16; no longer MYSX.13
- net PB9: no longer MYSX.14
Other:
- note added: "MysX 2.6 mysX Maple Mini 1 VRAW 2 3V3 3 VCCio 4 GND 5 PA9 6 PA10 7 RESET 8 PB1 9 PA0 10 PA8 11 PB6 12 PB7 13 PB10 14 PB11 15 PB0 16 PB8 17 PB5 18 PB4 19 PB3 20 PA15 21 PA2 22 PA3"
- note added: "Radio 1 alternativ"
- note added: "Radio1"
- note removed: "MysX 2.6 Pin/Arduino Port STM32 1 VRaw * 2 3V3 * 3 VCCio * 4 GND * 5 D1_DFM/TX PA9 6 D2_DTM/RX PA10 7 RST Reset 8 LEGACY_ID PB10 ??? 9 D3_INT PA0 (WakeUP) 10 D4_INT PA8 11 D5_PWM PB6 12 D6_PWM PB7 13 D7_SCL PB8 14 D8_SCA PB9 15 D9_A3 PA2 16 D10_A4 PA3 17 D11_MOSI PB5 18 D12_MISO PB4 19 D13_SCK PB3 20 D14_CS PA15 21 A5 PB0 22 A6 PB1"
- note removed: "Radio 0"
