File: MySensors-HM-easy-PCB-RFM-CC1101-RS485-NRF/5-GW-Sens-CAN-ProMicro/MySens-GWeasySensRS485-V01-040.sch (EAGLE design)
At the start: 24 parts, among them IC1 ATSHA204A, IC2 LD117ADT50TR, IC6 LM1117MPX-ADJ, X4 1751264

Commit message: Rework CAN
Parts:
- removed U$3: 2.1MMJACKTHM, adafruit:2.1MMJACKTHM
- added CH, CL: JUMPER-SMT_3_1-NC_TRACE_SILK, SparkFun-Jumpers:JUMPER-SMT_3_1-NC_TRACE_SILK
- added R3, R4: 680R, rcl:R-EU_R0805
- IC1: value ATSHA204A -> LM1117MPX-ADJ; device Sensor:ATSHA204A -> lm1117:LM1117MPX-ADJ
- renumbered JP10 to I2C
Connections:
- removed net 4: J4-1.4
- removed net 5: J4-1.5
- removed net N$2: J4-2.4
- removed net N$3: J4-2.5
- new net CANH: CL.1, J4-1.4, J4-2.4, X4-2.K
- new net CANL: CH.1, J4-1.5, J4-2.5, X4-3.K
- new net H: CL.2, R3.2, R6.1, U$1.CANH
- new net L: CH.2, R4.1, R6.2, U$1.CANL
- net 3V3: now also I2C.1, IC1.OUT, IC1.OUT1, SV2.2; no longer IC1.VCC
- net A: now also CH.3; no longer R6.1, U$1.CANH, X4-2.K
- net B: now also CL.3; no longer R6.2, U$1.CANL, X4-3.K
- net D7: no longer IC1.SDA
- net GND: now also IC1.ADJ, R4.2; no longer IC1.GND, U$3.RING
- net UREG: now also IC1.IN
- net VCC: now also R3.1; no longer I2C.1, SV2.2, X4-1.K
- net VIN: now also X4-1.K; no longer U$3.TIP
Other:
- note added: "1 Vraw (typically unregulated voltage, either from motherboard to daughterboard or vice versa) Motherboard should have a jumper to cut onboard Vraw source if daughterboard provides Vraw. Be sure to check motherboard constraints on Vraw before connecting a daughterboard that provides Vraw (for over voltage protection). Should be able to source at least 100mA and all boards are recommended to suppo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"
- note added: "Ext. Power Converters"
- note removed: "ATSHA204 authentication chip optional for MySensors"
- note removed: "Power Converters"
- moved on the sheet: C4, C6, F2, IC2, IC6, OPT3, R6, RAW1
