File: MySensors-HM-easy-PCB-RFM-CC1101-RS485-NRF/5-GW-Sens-RS485-CAN-ProMicro/MySens-GWeasySensRS485-V01-045.brd (EAGLE design)
At the start: 33 x 50 mm, 27 parts, among them IC1 LM1117MPX-ADJ, IC2 LD117ADT50TR, IC6 LM1117MPX-ADJ, X4 1751264

Commit message: CAN
Parts:
- added REG_BRIDGE: (no value), jumper:SJ
Connections:
- removed net VIN: F2.2, RAW1.1, X4.1
- new net UIN: C6.1, F2.1, IC1.3, IC2.3, IC6.3, RAW1.2, REG_BRIDGE.1, STEPDWN.3
- net IN: now also F2.2, RAW1.1, X4.1
- net UREG: now also REG_BRIDGE.2; no longer C6.1, F2.1, IC1.3, IC2.3, IC6.3, RAW1.2, STEPDWN.3
Routing:
- net UIN: track 0.00 -> 84.2 mm
- net UREG: track 94.2 -> 54.8 mm
- net IN: track 27.7 -> 44.6 mm, vias 0 -> 1
- net CANL: track 40.8 -> 51.2 mm
- net CANH: track 40.9 -> 51.0 mm
- net GND: track 150.6 -> 143.3 mm, vias 1 -> 24
- net VCC: track 123.0 -> 115.9 mm, vias 1 -> 2
- net D9: track 40.3 -> 45.8 mm, vias 0 -> 1
- net TX1: track 82.1 -> 76.6 mm, vias 0 -> 1
- net 3V3: track 38.5 -> 43.8 mm, vias 1 -> 2
- net D8: track 36.6 -> 31.3 mm
- net 2: track 13.9 -> 8.86 mm, vias 1 -> 0
- net D5: track 23.4 -> 28.3 mm, vias 0 -> 1
- net RX0: track 58.4 -> 63.3 mm
- net D2: track 32.0 -> 27.5 mm
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- added copper zone on layer 1, net GND
- added copper zone on layer 16, net GND
Other:
- board text added: "3v3"
- board text added: "A"
- board text added: "A0"
- board text added: "A1"
- board text added: "A2"
- board text added: "A3"
- board text added: "B"
- board text added: "D2"
- board text added: "D3"
- board text added: "D5"
- board text added: "D6"
- board text added: "D7"
- board text added: "D8"
- board text added: "D9"
- board text added: "MISO"
- board text added: "MOSI"
- board text added: "RST"
- board text added: "SCK"
- board text added: "SS"
