File: MySensors-HM-easy-PCB-RFM-CC1101-RS485-NRF/5-GW-Sens-RS485-CAN-ProMicro/MySens-GWeasySensRS485-V01-045.sch (EAGLE design)
At the start: 27 parts, among them IC1 LM1117MPX-ADJ, IC2 LD117ADT50TR, IC6 LM1117MPX-ADJ, X4 1751264

Commit message: CAN
Parts:
- added REG_BRIDGE: (no value), jumper:SJ
Connections:
- removed net VIN: F2.2, RAW1.1, X4-1.K
- new net UIN: C6.1, F2.1, IC1.IN, IC2.IN, IC6.IN, RAW1.2, REG_BRIDGE.1, STEPDWN.3
- net IN: now also F2.2, RAW1.1, X4-1.K
- net UREG: now also REG_BRIDGE.2; no longer C6.1, F2.1, IC1.IN, IC2.IN, IC6.IN, RAW1.2, STEPDWN.3
