File: MySensors-HM-easy-PCB-RFM-CC1101-RS485-NRF/5-GW-Sens-RS485-CAN-ProMicro/MySens-GWeasySensRS485-V03-062.brd (EAGLE design)
At the start: 33 x 50 mm, 27 parts, among them IC1 LM1117MPX-ADJ, IC2 LD117ADT50TR, IC6 LM1117MPX-ADJ, X4 1751264

Commit message: div
Parts:
- added R5: XKXR, rcl:R0805
- moved R2 4.74 mm to (26.0, 13.5), turned to 0 degrees
- moved R6 4.74 mm to (26.0, 10.3)
- moved U$1 4.20 mm to (17.8, 11.6)
- moved R3 4.05 mm to (10.2, 13.5), turned to 180 degrees
- moved IC2 4.00 mm to (29.3, 34.0)
- moved C4 4.00 mm to (23.1, 19.0)
- moved B1 4.00 mm to (15.0, 33.7)
- moved C3 4.00 mm to (16.5, 17.3)
- moved C6 4.00 mm to (1.89, 45.3)
- moved F2 4.00 mm to (3.81, 20.5)
- moved I2C 4.00 mm to (3.17, 33.2)
- moved J4 4.00 mm to (16.5, 2.73)
- moved JP1 4.00 mm to (5.08, 13.5)
- moved JP3 4.00 mm to (2.54, 13.5)
- moved OPT3 4.00 mm to (16.5, 5.91)
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Connections:
- net A: now also R3.2, R5.1, R6.1, U$1.CANH; no longer R4.1, R6.2, U$1.CANL
- net B: now also R4.1, R6.2, U$1.CANL; no longer R3.2, R6.1, U$1.CANH
- net GND: now also R5.2
Routing:
- net A: track 33.4 -> 52.5 mm
- net VCC: track 132.1 -> 115.0 mm, vias 0 -> 2
- net 3V3: track 75.9 -> 59.0 mm
- net D3: track 21.5 -> 36.3 mm, vias 0 -> 1
- net A5: track 54.5 -> 40.1 mm
- net TX1: track 54.3 -> 67.4 mm
- net D13_SCK: track 49.1 -> 61.0 mm, vias 1 -> 0
- net D12_MISO: track 46.7 -> 57.6 mm
- net D5: track 33.9 -> 26.9 mm
- net D2: track 32.5 -> 25.8 mm, vias 1 -> 2
- net GND: track 168.5 -> 163.5 mm, vias 21 -> 18
- net RX0: track 53.5 -> 49.8 mm
- net B: track 39.7 -> 36.3 mm
- net RESET: track 44.1 -> 46.9 mm, vias 1 -> 0
- net CANH: track 16.8 -> 19.3 mm
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Other:
- board text added: "ProMicro easySens V0.3CAN"
- board text removed: "ProMicro easySens V0.2CAN"
