File: Experimental/ESP32/MySens-easyESP32-003.brd (EAGLE design)
At the start: 74 x 34 mm, 48 parts, among them IC2 TP4056, IC5 LD117ADT50TR, IC6 LM1117MPX-ADJ, U2 RFM69HCW, U3 ESP-WROOM-32

Commit message: ESP32
Parts:
- added JP1: JUMPER-SMT_2_NC_PASTE_NO-SILK, SparkFun-Jumpers:SMT-JUMPER_2_NC_PASTE_NO-SILK
- added U1: 3.3V, SparkFun-IC-Power:SOT23-5
- added U4: RT9013-XXXB, v-reg:SOT23-5
Connections:
- new net MAYBE_IO5: CC0.GDO2, JP1.2
- net GND: now also U4.2
- net IO5: now also JP1.1; no longer CC0.GDO2
Changed lines of the file:
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@@
 <element name="J1" library="SparkFun-Connectors" package="1X02_XTRA_BIG" value="" x="-2.54" y="-82.55"/>
 <element name="J2" library="SparkFun-Connectors" package="1X02_XTRA_BIG" value="" x="-11.43" y="-88.9"/>
+<element name="JP1" library="SparkFun-Jumpers" package="SMT-JUMPER_2_NC_PASTE_NO-SILK" value="JUMPER-SMT_2_NC_PASTE_NO-SILK" x="-20.32" y="-93.98"/>
+<element name="U1" library="SparkFun-IC-Power" package="SOT23-5" value="3.3V" x="-24.13" y="-80.645">
+<attribute name="PROD_ID" value="VREG-12457" x="-24.13" y="-80.645" size="1.778" layer="27" display="off"/>
+</element>
+<element name="U4" library="v-reg" package="SOT23-5" value="RT9013-XXXB" x="-30.48" y="-80.645"/>
 </elements>
 <signals>
@@
 <contactref element="J1" pad="1"/>
 <contactref element="IC2" pad="1"/>
-<wire x1="86.12" y1="12.7" x2="36.195" y2="4.445" width="0" layer="19" extent="1-1"/>
-<wire x1="78.5" y1="15.11" x2="86.12" y2="12.7" width="0" layer="19" extent="16-16"/>
-<wire x1="72.785" y1="17.91" x2="78.5" y2="15.11" width="0" layer="19" extent="16-16"/>
-<wire x1="61.675" y1="3.175" x2="72.785" y2="17.91" width="0" layer="19" extent="16-16"/>
-<wire x1="53.656" y1="3.3" x2="61.675" y2="3.175" width="0" layer="19" extent="16-16"/>
-<wire x1="53.735" y1="15.24" x2="53.656" y2="3.3" width="0" layer="19" extent="16-16"/>
-<wire x1="35.04" y1="-11.135" x2="53.735" y2="15.24" width="0" layer="19" extent="16-16"/>
-<wire x1="21.47" y1="28.35" x2="35.04" y2="-11.135" width="0" layer="19" extent="16-16"/>
-<wire x1="21.47" y1="14.35" x2="21.47" y2="28.35" width="0" layer="19" extent="16-16"/>
-<wire x1="10.19375" y1="12.8725" x2="21.47" y2="14.35" width="0" layer="19" extent="16-16"/>
+<contactref element="U4" pad="2"/>
+<wire x1="-15.45" y1="-83.185" x2="-30.48" y2="-81.9451" width="0" layer="19" extent="1-1"/>
+<wire x1="-15.45" y1="-80.645" x2="-15.45" y2="-83.185" width="0" layer="19" extent="1-1"/>
+<wire x1="-8.89" y1="-88.9" x2="-15.45" y2="-83.185" width="0" layer="19" extent="1-1"/>
+<wire x1="-5.08" y1="-82.55" x2="-8.89" y2="-88.9" width="0" layer="19" extent="1-1"/>
+<wire x1="-3.658" y1="-95.25" x2="-8.89" y2="-88.9" width="0" layer="19" extent="1-1"/>
+<wire x1="-12.7" y1="-67.31" x2="-15.45" y2="-80.645" width="0" layer="19" extent="1-1"/>
+<wire x1="-2.54" y1="-67.31" x2="-12.7" y2="-67.31" width="0" layer="19" extent="1-1"/>
+<wire x1="-5.45" y1="-52.07" x2="-2.54" y2="-67.31" width="0" layer="19" extent="1-1"/>
+<wire x1="-3.27" y1="-41.91" x2="-5.45" y2="-52.07" width="0" layer="19" extent="1-1"/>
+<wire x1="-10.89" y1="-41.91" x2="-3.27" y2="-41.91" width="0" layer="19" extent="1-1"/>
+<wire x1="-15.24" y1="-47.498" x2="-10.89" y2="-41.91" width="0" layer="19" extent="1-1"/>
+<wire x1="4.23" y1="-39.37" x2="-3.27" y2="-41.91" width="0" layer="19" extent="1-1"/>
+<wire x1="11.01" y1="-39.37" x2="4.23" y2="-39.37" width="0" layer="19" extent="1-1"/>
+<wire x1="-0.875" y1="-11.115" x2="4.23" y2="-39.37" width="0" layer="19" extent="1-16"/>
+<wire x1="7.67" y1="5.325" x2="-0.875" y2="-11.115" width="0" layer="19" extent="16-16"/>
+<wire x1="5" y1="8.78" x2="7.67" y2="5.325" width="0" layer="19" extent="1-16"/>
+<wire x1="7.67" y1="10.405" x2="5" y2="8.78" width="0" layer="19" extent="1-16"/>
+<wire x1="2.032" y1="7.62" x2="5" y2="8.78" width="0" layer="19" extent="1-16"/>
+<wire x1="2.032" y1="7.62" x2="2.032" y2="7.62" width="0" layer="19" extent="1-16"/>
+<wire x1="10.19375" y1="12.8725" x2="7.67" y2="10.405" width="0" layer="19" extent="16-16"/>
 <wire x1="10.19375" y1="16.71375" x2="10.19375" y2="12.8725" width="0" layer="19" extent="16-16"/>
+<wire x1="12.7" y1="17.78" x2="10.19375" y2="16.71375" width="0" layer="19" extent="1-16"/>
 <wire x1="6.47" y1="16.35" x2="10.19375" y2="16.71375" width="0" layer="19" extent="16-16"/>
 <wire x1="2.032" y1="17.78" x2="6.47" y2="16.35" width="0" layer="19" extent="1-16"/>
 <wire x1="2.032" y1="17.78" x2="2.032" y2="17.78" width="0" layer="19" extent="1-16"/>
-<wire x1="2.032" y1="12.7" x2="2.032" y2="17.78" width="0" layer="19" extent="1-1"/>
+<wire x1="2.032" y1="12.7" x2="5" y2="8.78" width="0" layer="19" extent="1-16"/>
 <wire x1="2.032" y1="12.7" x2="2.032" y2="12.7" width="0" layer="19" extent="1-16"/>
-<wire x1="26.67" y1="13.905" x2="10.19375" y2="16.71375" width="0" layer="19" extent="1-16"/>
-<wire x1="42.2812" y1="-8.14" x2="21.47" y2="14.35" width="0" layer="19" extent="16-16"/>
+<wire x1="21.47" y1="14.35" x2="12.7" y2="17.78" width="0" layer="19" extent="1-16"/>
+<wire x1="23" y1="12.065" x2="21.47" y2="14.35" width="0" layer="19" extent="1-16"/>
+<wire x1="26.67" y1="13.905" x2="23" y2="12.065" width="0" layer="19" extent="1-16"/>
+<wire x1="5" y1="26.78" x2="2.032" y2="17.78" width="0" layer="19" extent="1-1"/>
+<wire x1="36.195" y1="4.445" x2="26.67" y2="13.905" width="0" layer="19" extent="16-16"/>
+<wire x1="21.47" y1="28.35" x2="12.7" y2="17.78" width="0" layer="19" extent="1-16"/>
+<wire x1="42.2812" y1="-8.14" x2="36.195" y2="4.445" width="0" layer="19" extent="16-16"/>
+<wire x1="35.04" y1="-11.135" x2="42.2812" y2="-8.14" width="0" layer="19" extent="16-16"/>
 <wire x1="50.56" y1="-12.065" x2="42.2812" y2="-8.14" width="0" layer="19" extent="16-16"/>
-<wire x1="7.67" y1="5.325" x2="21.47" y2="28.35" width="0" layer="19" extent="1-16"/>
-<wire x1="7.67" y1="10.405" x2="7.67" y2="5.325" width="0" layer="19" extent="1-1"/>
-<wire x1="2.032" y1="7.62" x2="7.67" y2="5.325" width="0" layer="19" extent="1-1"/>
-<wire x1="2.032" y1="7.62" x2="2.032" y2="7.62" width="0" layer="19" extent="1-16"/>
-<wire x1="2.032" y1="12.7" x2="2.032" y2="7.62" width="0" layer="19" extent="1-1"/>
-<wire x1="2.032" y1="12.7" x2="2.032" y2="12.7" width="0" layer="19" extent="1-16"/>
-<wire x1="-0.875" y1="-11.115" x2="26.67" y2="13.905" width="0" layer="19" extent="1-16"/>
-<wire x1="47.665" y1="50.54" x2="2.032" y2="7.62" width="0" layer="19" extent="1-1"/>
-<wire x1="48.731" y1="50.571" x2="47.665" y2="50.54" width="0" layer="19" extent="1-1"/>
-<wire x1="64.77" y1="50.165" x2="48.731" y2="50.571" width="0" layer="19" extent="1-1"/>
-<wire x1="5" y1="8.78" x2="2.032" y2="12.7" width="0" layer="19" extent="1-1"/>
-<wire x1="12.7" y1="17.78" x2="5" y2="8.78" width="0" layer="19" extent="1-1"/>
-<wire x1="23" y1="12.065" x2="12.7" y2="17.78" width="0" layer="19" extent="1-1"/>
-<wire x1="5" y1="26.78" x2="12.7" y2="17.78" width="0" layer="19" extent="1-1"/>
-<wire x1="4.23" y1="-39.37" x2="5" y2="26.78" width="0" layer="19" extent="1-1"/>
-<wire x1="11.01" y1="-39.37" x2="4.23" y2="-39.37" width="0" layer="19" extent="1-1"/>
-<wire x1="-3.27" y1="-41.91" x2="4.23" y2="-39.37" width="0" layer="19" extent="1-1"/>
-<wire x1="-10.89" y1="-41.91" x2="-3.27" y2="-41.91" width="0" layer="19" extent="1-1"/>
-<wire x1="-15.24" y1="-47.498" x2="-10.89" y2="-41.91" width="0" layer="19" extent="1-1"/>
-<wire x1="-5.45" y1="-52.07" x2="-3.27" y2="-41.91" width="0" layer="19" extent="1-1"/>
-<wire x1="-2.54" y1="-67.31" x2="-5.45" y2="-52.07" width="0" layer="19" extent="1-1"/>
-<wire x1="-12.7" y1="-67.31" x2="-2.54" y2="-67.31" width="0" layer="19" extent="1-1"/>
-<wire x1="-15.45" y1="-80.645" x2="-12.7" y2="-67.31" width="0" layer="19" extent="1-1"/>
-<wire x1="-15.45" y1="-83.185" x2="-15.45" y2="-80.645" width="0" layer="19" extent="1-1"/>
-<wire x1="-8.89" y1="-88.9" x2="-15.45" y2="-83.185" width="0" layer="19" extent="1-1"/>
-<wire x1="-5.08" y1="-82.55" x2="-8.89" y2="-88.9" width="0" layer="19" extent="1-1"/>
-<wire x1="-3.658" y1="-95.25" x2="-8.89" y2="-88.9" width="0" layer="19" extent="1-1"/>
-<wire x1="-7.935" y1="59.055" x2="-0.875" y2="-11.115" width="0" layer="19" extent="1-16"/>
+<wire x1="53.656" y1="3.3" x2="50.56" y2="-12.065" width="0" layer="19" extent="16-16"/>
+<wire x1="61.675" y1="3.175" x2="53.656" y2="3.3" width="0" layer="19" extent="16-16"/>
+<wire x1="53.735" y1="15.24" x2="53.656" y2="3.3" width="0" layer="19" extent="16-16"/>
+<wire x1="72.785" y1="17.91" x2="61.675" y2="3.175" width="0" layer="19" extent="16-16"/>
+<wire x1="78.5" y1="15.11" x2="72.785" y2="17.91" width="0" layer="19" extent="16-16"/>
+<wire x1="86.12" y1="12.7" x2="78.5" y2="15.11" width="0" layer="19" extent="16-16"/>
+<wire x1="64.77" y1="50.165" x2="72.785" y2="17.91" width="0" layer="19" extent="16-16"/>
+<wire x1="48.731" y1="50.571" x2="64.77" y2="50.165" width="0" layer="19" extent="1-1"/>
+<wire x1="47.665" y1="50.54" x2="48.731" y2="50.571" width="0" layer="19" extent="1-1"/>
+<wire x1="-7.935" y1="59.055" x2="5" y2="26.78" width="0" layer="19" extent="1-1"/>
 </signal>
 <signal name="VCC" class="1">
@@
 <signal name="IO5">
 <contactref element="U3" pad="29"/>
-<contactref element="CC0" pad="GDO2"/>
-<wire x1="16.43" y1="26.78" x2="26.67" y2="5.905" width="0" layer="19" extent="1-1"/>
+<contactref element="JP1" pad="1"/>
+<wire x1="16.43" y1="26.78" x2="-20.7264" y2="-93.98" width="0" layer="19" extent="1-1"/>
 </signal>
 <signal name="IO15">
@@
 <contactref element="MYSX" pad="15"/>
 </signal>
+<signal name="MAYBE_IO5">
+<contactref element="CC0" pad="GDO2"/>
+<contactref element="JP1" pad="2"/>
+<wire x1="26.67" y1="5.905" x2="-19.9136" y2="-93.98" width="0" layer="19" extent="1-16"/>
+</signal>
 </signals>
