File: Experimental/ESP32/MySens-easyESP32-003.sch (EAGLE design)
At the start: 48 parts, among them IC2 TP4056, IC5 LD117ADT50TR, IC6 LM1117MPX-ADJ, U2 RFM69HCW, U3 ESP-WROOM-32

Commit message: ESP32
Parts:
- added JP1: JUMPER-SMT_2_NC_PASTE_NO-SILK, SparkFun-Jumpers:JUMPER-SMT_2_NC_PASTE_NO-SILK
- added U1: 3.3V, SparkFun-IC-Power:V_REG_AP2112K-3.3V
- added U4: RT9013-XXXB, v-reg:RT9013-XXXB
Connections:
- new net MAYBE_IO5: CC0.GDO2, JP1.2
- net IO5: now also JP1.1; no longer CC0.GDO2
Other:
- note added: "Kann Weg bei Platzmangel"
- note added: "Wenn man die Pins von dem MYSx Stecker: 3.3V, GND, RX, TX, EN und GPIO00 nimmt und einen Standad USB Programmer (z.B. einen FDDI um 1,60€) nimmt und den EN auf RTS und GPIO00 auf DTR verbindet. Dann setzt der Flasher den Chip automatisch in den Flash Mode, führt den Flash durch und macht den Reset und started den geflashten Sketch."
Changed lines of the file:
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@@
 <part name="GND17" library="supply1" deviceset="GND" device=""/>
 <part name="J2" library="SparkFun-Connectors" deviceset="CONN_02" device="PTH4"/>
+<part name="JP1" library="SparkFun-Jumpers" deviceset="JUMPER-SMT_2_NC_PASTE" device="_NO-SILK"/>
+<part name="U1" library="SparkFun-IC-Power" deviceset="V_REG_AP2112" device="K-3.3V" value="3.3V"/>
+<part name="U4" library="v-reg" deviceset="RT9013-XXX" device="B"/>
 </parts>
 <sheets>
@@
 <text x="25.4" y="-149.86" size="1.778" layer="97">Regulator</text>
 <text x="-127" y="-172.72" size="1.778" layer="97">Div</text>
-<text x="-38.1" y="-43.18" size="1.778" layer="97">mysX	ESP32
-1	VRAW
-2	3V3
-3	VCCio
-4	GND
-5	TXD0
-6	RXD0
-7	EN
-8	IO27
-9	IO0
-10	IO2
-11	IO4
-12	IO25
-13	IO22
-14	IO21
-15	SENSOR_VN
-16	IO15
-17	IO13
-18	IO12
-19	IO14
-20	IO26
-21	IO34
-22	IO35</text>
+<text x="-38.1" y="-43.18" size="1.778" layer="97">mysX ESP32
+1 VRAW
+2 3V3
+3 VCCio
+4 GND
+5 TXD0
+6 RXD0
+7 EN
+8 IO27
+9 IO0
+10 IO2
+11 IO4
+12 IO25
+13 IO22
+14 IO21
+15 SENSOR_VN
+16 IO15
+17 IO13
+18 IO12
+19 IO14
+20 IO26
+21 IO34
+22 IO35</text>
 <text x="40.64" y="-165.1" size="1.778" layer="97" rot="R270">PB0 auch am mysX</text>
 <text x="55.88" y="67.31" size="3.81" layer="95" ratio="15">Radio1</text>
@@
 <text x="181.61" y="54.61" size="3.81" layer="95" ratio="15">CC1101</text>
 <text x="88.9" y="149.86" size="6.4516" layer="102">Achtung</text>
-<circle x="170.18" y="27.94" radius="2.54" width="0.1524" layer="102"/>
+<circle x="152.4" y="27.94" radius="2.54" width="0.1524" layer="102"/>
 <text x="137.16" y="55.88" size="5.08" layer="102">???? io5 ???</text>
+<wire x1="15.24" y1="73.66" x2="15.24" y2="27.94" width="0.1524" layer="97" style="shortdash"/>
+<wire x1="15.24" y1="27.94" x2="43.18" y2="27.94" width="0.1524" layer="97" style="shortdash"/>
+<wire x1="43.18" y1="27.94" x2="43.18" y2="78.74" width="0.1524" layer="97" style="shortdash"/>
+<wire x1="43.18" y1="78.74" x2="15.24" y2="78.74" width="0.1524" layer="97" style="shortdash"/>
+<wire x1="15.24" y1="78.74" x2="15.24" y2="73.66" width="0.1524" layer="97" style="shortdash"/>
+<text x="15.24" y="25.4" size="1.778" layer="97">Kann Weg bei Platzmangel</text>
+<text x="-63.5" y="-55.88" size="1.778" layer="97">Wenn man die Pins von dem MYSx Stecker: 3.3V, GND, RX, TX, EN und GPIO00
+nimmt und einen Standad USB Programmer (z.B. einen FDDI um 1,60€) nimmt und den
+EN auf RTS und GPIO00 auf DTR verbindet. Dann setzt der Flasher den Chip automatisch in den Flash Mode, führt den Flash durch und
+macht den Reset und started den geflashten Sketch.</text>
 </plain>
 <instances>
@@
 <instance part="GND17" gate="1" x="-198.12" y="-27.94" rot="R270"/>
 <instance part="J2" gate="G$1" x="-154.94" y="-38.1" rot="R180"/>
+<instance part="JP1" gate="G$1" x="162.56" y="27.94" smashed="yes">
+<attribute name="NAME" x="160.02" y="30.48" size="1.778" layer="95" font="vector"/>
+</instance>
+<instance part="U1" gate="G$1" x="-30.48" y="-119.38"/>
+<instance part="U4" gate="G$1" x="-30.48" y="-96.52"/>
 </instances>
 <busses>
@@
 </segment>
 <segment>
-<pinref part="CC0" gate="G$1" pin="GDO2"/>
-<wire x1="167.64" y1="27.94" x2="175.26" y2="27.94" width="0.1524" layer="91"/>
-<label x="168.91" y="27.94" size="1.778" layer="95"/>
+<pinref part="JP1" gate="G$1" pin="1"/>
+<wire x1="157.48" y1="27.94" x2="149.86" y2="27.94" width="0.1524" layer="91"/>
+<label x="149.86" y="27.94" size="1.778" layer="95"/>
 </segment>
 </net>
@@
 </segment>
 </net>
+<net name="MAYBE_IO5" class="0">
+<segment>
+<pinref part="CC0" gate="G$1" pin="GDO2"/>
+<pinref part="JP1" gate="G$1" pin="2"/>
+<wire x1="167.64" y1="27.94" x2="175.26" y2="27.94" width="0.1524" layer="91"/>
+</segment>
+</net>
