File: Experimental/ESP32/50x33/MySens-easyESP32b-007c.brd (EAGLE design)
At the start: 33 x 50 mm, 22 parts, among them U2 RFM69HCW, U3 ESP-WROOM-32

Commit message: ESP32 SMD
Parts:
- moved R2 28.9 mm to (21.0, 26.7), turned to 0 degrees
- moved JP1 20.0 mm to (31.5, 37.5), turned to 270 degrees
- moved C6 6.38 mm to (3.17, 48.3)
- moved R6 3.86 mm to (10.8, 48.3)
- moved R3 3.86 mm to (10.8, 24.1)
- moved C9 2.62 mm to (16.5, 24.1)
- moved C2 1.42 mm to (6.99, 26.7)
- moved U3 1.27 mm to (16.5, 41.3)
- moved TP4056 1.16 mm to (14.3, 38.3), turned to 180 degrees
- moved R7 0.90 mm to (3.17, 29.2), turned to 0 degrees
- moved AP2112 0.90 mm to (3.17, 35.6)
- moved F2 0.64 mm to (1.91, 17.8)
- moved R1 0.64 mm to (1.91, 22.9)
- moved U2 0.63 mm to (13.3, 12.1)
Routing:
- net MAYBE_IO5: track 1.88 -> 47.5 mm, vias 0 -> 2
- net IO5: track 34.6 -> 6.23 mm
- net IN++: track 43.9 -> 16.0 mm
- net B+: track 42.9 -> 68.3 mm, vias 3 -> 0
- net B-: track 32.0 -> 53.1 mm, vias 3 -> 1
- net IO14: track 25.6 -> 45.9 mm, vias 1 -> 2
- net IO27: track 37.2 -> 55.3 mm, vias 2 -> 1
- net IO26: track 24.5 -> 40.4 mm, vias 1 -> 3
- net IO12: track 23.1 -> 35.9 mm, vias 1 -> 2
- net EN: track 78.5 -> 67.5 mm, vias 4 -> 2
- net IO17: track 49.6 -> 60.0 mm, vias 2 -> 5
- net IO25: track 43.8 -> 34.1 mm, vias 1 -> 3
- net UREG: track 82.3 -> 73.1 mm, vias 3 -> 1
- net IN-: track 53.1 -> 44.0 mm
- net TXD0: track 41.4 -> 48.1 mm, vias 0 -> 2
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- added copper zone on layer 1, net GND
- added copper zone on layer 16, net GND
