File: Experimental/ESP32/50x33/MySens-easyESP32b-012.brd (EAGLE design)
At the start: 33 x 50 mm, 23 parts, among them U2 RFM69HCW, U3 ESP-WROOM-32

Commit message: ESP32
Routing:
- net GND: vias 3 -> 16
- added copper zone on layer 1, net GND
- added copper zone on layer 16, net GND
Other:
- board text added: "(C) www.neuby.de"
- board text added: "3V3"
- board text added: "ANT(RFM)"
- board text added: "B+"
- board text added: "B-"
- board text added: "Bat-"
- board text added: "EN"
- board text added: "ESP32 MysX V0.1"
- board text added: "IN+"
- board text added: "IN-"
- board text added: "IO0"
- board text added: "IO12"
- board text added: "IO13"
- board text added: "IO15"
- board text added: "IO2"
- board text added: "IO21"
- board text added: "IO22"
- board text added: "IO25"
- board text added: "IO26"
- board text added: "IO27"
- board text added: "IO34"
- board text added: "IO35"
- board text added: "IO4"
- board text added: "RX"
- board text added: "TCD0"
- board text added: "VIN"
- board text added: "VN"
- board text removed: "5V"
- board text removed: "PluepillGW V01 RS485, RFM69, RFM95"
- board text removed: "SDA"
- board text removed: "SDL"
- board text removed: "easyGW BluePill 0.2 RS485, RFM69, RFM95"
Changed lines of the file:
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@@
 <?xml version="1.0" encoding="utf-8"?>
 <!DOCTYPE eagle SYSTEM "eagle.dtd">
-<eagle version="7.6.0">
+<eagle version="9.1.0">
 <drawing>
 <settings>
 <setting alwaysvectorfont="no"/>
+<setting keepoldvectorfont="yes"/>
 <setting verticaltext="up"/>
 </settings>
-<grid distance="50" unitdist="mil" unit="mil" style="lines" multiple="1" display="yes" altdistance="0.1" altunitdist="mm" altunit="mm"/>
+<grid distance="10" unitdist="mil" unit="mil" style="lines" multiple="1" display="yes" altdistance="0.1" altunitdist="mm" altunit="mm"/>
 <layers>
 <layer number="1" name="Top" color="4" fill="1" visible="yes" active="yes"/>
@@
 <plain>
 <text x="45.287" y="65.485" size="0.6096" layer="25"></text>
-<text x="50.56" y="22.86" size="0.6096" layer="25" font="vector" rot="R90">SDA</text>
-<text x="50.56" y="27.94" size="0.6096" layer="25" font="vector" rot="R90">GND</text>
-<text x="50.56" y="25.4" size="0.6096" layer="25" font="vector" rot="R90">SDL</text>
-<text x="50.56" y="30.48" size="0.6096" layer="25" font="vector" rot="R90">VCC</text>
-<text x="85.103" y="33.256" size="1.016" layer="25" font="vector" rot="R180">easyGW BluePill 0.2
-RS485, RFM69, RFM95</text>
-<text x="75.563" y="26.398" size="1.016" layer="26" font="vector" rot="MR0">PluepillGW V01
-RS485, RFM69, RFM95</text>
-<text x="87.489" y="11.303" size="0.6096" layer="25" font="vector" rot="R270">5V</text>
-<text x="87.489" y="18.923" size="0.6096" layer="25" font="vector" rot="R270">5V</text>
-<text x="87.489" y="13.843" size="0.6096" layer="25" font="vector" rot="R270">GND</text>
-<text x="87.489" y="16.383" size="0.6096" layer="25" font="vector" rot="R270">UREG</text>
+<text x="4.431" y="14.605" size="0.6096" layer="25" font="vector" rot="R270">VIN</text>
+<text x="4.431" y="12.319" size="0.6096" layer="25" font="vector" rot="R270">GND</text>
 <wire x1="-3" y1="-1.5" x2="-3" y2="35.5" width="0.1" layer="49"/>
 <wire x1="-3" y1="35.5" x2="-1.5" y2="37" width="0.1" layer="49" curve="-90"/>
@@
 <wire x1="33" y1="0" x2="33" y2="50" width="0" layer="20"/>
 <wire x1="0" y1="50" x2="33" y2="50" width="0" layer="20"/>
+<text x="23.368" y="2.794" size="1.778" layer="26" rot="MR90">ESP32 MysX V0.1</text>
+<text x="22.86" y="25.4" size="1.27" layer="25" rot="R270">(C) www.neuby.de</text>
+<text x="4.431" y="9.525" size="0.6096" layer="25" font="vector" rot="R270">Bat-</text>
+<text x="4.431" y="6.985" size="0.6096" layer="25" font="vector" rot="R270">B+</text>
+<text x="27.305" y="0.621" size="0.6096" layer="25" font="vector">3V3</text>
+<text x="32.653" y="1.905" size="0.6096" layer="25" font="vector" rot="R90">VIN</text>
+<text x="32.653" y="4.191" size="0.6096" layer="25" font="vector" rot="R90">VCC</text>
+<text x="32.653" y="6.477" size="0.6096" layer="25" font="vector" rot="R90">TCD0</text>
+<text x="32.653" y="9.779" size="0.6096" layer="25" font="vector" rot="R90">EN</text>
+<text x="32.653" y="12.065" size="0.6096" layer="25" font="vector" rot="R90">IO0</text>
+<text x="32.653" y="14.605" size="0.6096" layer="25" font="vector" rot="R90">IO4</text>
+<text x="32.117" y="21.209" size="0.6096" layer="25" font="vector" rot="R270">VN</text>
+<text x="32.653" y="17.145" size="0.6096" layer="25" font="vector" rot="R90">IO22</text>
+<text x="26.543" y="5.983" size="0.6096" layer="25" font="vector" rot="R180">GND</text>
+<text x="25.767" y="8.001" size="0.6096" layer="25" font="vector" rot="R270">RX</text>
+<text x="25.767" y="10.795" size="0.6096" layer="25" font="vector" rot="R270">IO27</text>
+<text x="25.767" y="13.335" size="0.6096" layer="25" font="vector" rot="R270">IO2</text>
+<text x="25.767" y="15.875" size="0.6096" layer="25" font="vector" rot="R270">IO25</text>
+<text x="25.767" y="18.923" size="0.6096" layer="25" font="vector" rot="R270">IO21</text>
+<text x="25.767" y="21.209" size="0.6096" layer="25" font="vector" rot="R270">IO15</text>
+<text x="25.767" y="24.003" size="0.6096" layer="25" font="vector" rot="R270">IO12</text>
+<text x="25.767" y="26.543" size="0.6096" layer="25" font="vector" rot="R270">IO26</text>
+<text x="25.767" y="29.337" size="0.6096" layer="25" font="vector" rot="R270">IO35</text>
+<text x="32.117" y="23.495" size="0.6096" layer="25" font="vector" rot="R270">IO13</text>
+<text x="32.117" y="26.035" size="0.6096" layer="25" font="vector" rot="R270">IO4</text>
+<text x="32.117" y="28.829" size="0.6096" layer="25" font="vector" rot="R270">IO34</text>
+<text x="4.826" y="43.688" size="1.778" layer="26">IN-</text>
+<text x="4.826" y="30.48" size="1.778" layer="26">IN+</text>
+<text x="28.194" y="43.434" size="1.778" layer="26">GND</text>
+<text x="27.94" y="40.386" size="1.778" layer="26">B-</text>
+<text x="28.448" y="32.766" size="1.778" layer="26">B+</text>
+<text x="28.194" y="29.972" size="1.016" layer="26">UREG</text>
+<text x="1.27" y="45.72" size="0.8128" layer="26" rot="R90">IN-</text>
+<text x="1.27" y="28.194" size="0.8128" layer="26" rot="R90">IN+</text>
+<text x="6.096" y="19.304" size="0.8128" layer="25" rot="R90">VCC</text>
+<text x="8.128" y="19.304" size="0.8128" layer="25" rot="R90">GND</text>
+<text x="6.209" y="10.541" size="0.6096" layer="25" font="vector" rot="R270">ANT(RFM)</text>
 </plain>
 <attributes>
@@
 <param name="dpMaxLengthDifference" value="10mm"/>
 <param name="dpGapFactor" value="2.5"/>
-<param name="checkGrid" value="0"/>
 <param name="checkAngle" value="0"/>
 <param name="checkFont" value="1"/>
 <param name="checkRestrict" value="0"/>
+<param name="checkStop" value="0"/>
+<param name="checkValues" value="0"/>
+<param name="checkNames" value="1"/>
+<param name="checkWireStubs" value="1"/>
+<param name="checkPolygonWidth" value="0"/>
 <param name="useDiameter" value="13"/>
 <param name="maxErrors" value="50"/>
@@
 <element name="ANT2" library="pinhead" package="1X01" value="" x="13.97" y="1.905" rot="MR0"/>
 <element name="R7" library="rcl" package="M0805" value="100k" x="3.175" y="29.21"/>
-<element name="R5" library="rcl" package="R0603" value="10k" x="25.4" y="3.81" rot="R270"/>
+<element name="R5" library="rcl" package="R0603" value="10k" x="25.4" y="3.81" smashed="yes" rot="R270">
+<attribute name="NAME" x="22.987" y="4.445" size="1.27" layer="25" rot="R270"/>
+<attribute name="VALUE" x="23.495" y="4.445" size="1.27" layer="27" rot="R270"/>
+</element>
 </elements>
 <signals>
@@
 <wire x1="20.335" y1="19.565" x2="20.335" y2="21.547609375" width="0.4572" layer="1"/>
 <wire x1="27.94" y1="5.08" x2="27.94" y2="6.324609375" width="0.4572" layer="1"/>
+<polygon width="0.1524" layer="1">
+<vertex x="1.27" y="1.27"/>
+<vertex x="1.27" y="44.45"/>
+<vertex x="31.75" y="44.45"/>
+<vertex x="31.75" y="1.27"/>
+</polygon>
+<polygon width="0.1524" layer="16">
+<vertex x="1.27" y="1.27"/>
+<vertex x="1.27" y="44.45"/>
+<vertex x="31.75" y="44.45"/>
+<vertex x="31.75" y="1.27"/>
+</polygon>
+<via x="6.35" y="8.89" extent="1-16" drill="0.35" shape="square"/>
+<via x="6.35" y="15.24" extent="1-16" drill="0.35" shape="square"/>
+<via x="6.35" y="12.7" extent="1-16" drill="0.35" shape="square"/>
+<via x="11.43" y="15.24" extent="1-16" drill="0.35" shape="square"/>
+<via x="12.7" y="12.7" extent="1-16" drill="0.35" shape="square"/>
+<via x="13.97" y="10.16" extent="1-16" drill="0.35" shape="square"/>
+<via x="10.16" y="7.62" extent="1-16" drill="0.35" shape="square"/>
+<via x="22.86" y="3.81" extent="1-16" drill="0.35" shape="square"/>
+<via x="24.13" y="7.62" extent="1-16" drill="0.35" shape="square"/>
+<via x="25.4" y="13.97" extent="1-16" drill="0.35" shape="square"/>
+<via x="24.13" y="20.32" extent="1-16" drill="0.35" shape="square"/>
+<via x="17.78" y="27.94" extent="1-16" drill="0.35" shape="square"/>
+<via x="5.08" y="39.37" extent="1-16" drill="0.35" shape="square"/>
+<wire x1="16.415790625" y1="25.36261875" x2="17.78" y2="27.94" width="0" layer="19" extent="1-1"/>
+<wire x1="6.35" y1="15.24" x2="8.335" y2="15.582390625" width="0" layer="19" extent="1-1"/>
+<wire x1="10.16" y1="7.62" x2="11.185" y2="5.672809375" width="0" layer="19" extent="16-16"/>
+<wire x1="6.35" y1="12.7" x2="6.35" y2="15.24" width="0" layer="19" extent="1-1"/>
+<wire x1="5.08" y1="39.37" x2="2.513459375" y2="39.405340625" width="0" layer="19" extent="16-16"/>
+<wire x1="24.13" y1="7.62" x2="26.28038125" y2="5.495009375" width="0" layer="19" extent="16-16"/>
+<wire x1="11.43" y1="15.24" x2="8.335" y2="15.582390625" width="0" layer="19" extent="1-1"/>
+<wire x1="12.7" y1="12.7" x2="11.43" y2="15.24" width="0" layer="19" extent="1-1"/>
+<wire x1="13.97" y1="10.16" x2="12.7" y2="12.7" width="0" layer="19" extent="1-1"/>
+<wire x1="22.86" y1="3.81" x2="26.28038125" y2="5.495009375" width="0" layer="19" extent="16-16"/>
+<wire x1="6.35" y1="8.89" x2="6.35" y2="12.7" width="0" layer="19" extent="1-1"/>
+<wire x1="24.13" y1="20.32" x2="20.335" y2="19.565" width="0" layer="19" extent="1-1"/>
+<wire x1="25.4" y1="13.97" x2="20.335" y2="13.46288125" width="0" layer="19" extent="1-1"/>
 </signal>
 <signal name="VCC" class="1">
@@
 <wire x1="1.905" y1="19.18" x2="1.905" y2="20.10566875" width="0.4064" layer="16"/>
 </signal>
-<signal name="N$3">
-</signal>
-<signal name="N$6" class="1">
-</signal>
 </signals>
+<mfgpreviewcolors>
+<mfgpreviewcolor name="soldermaskcolor" color="0xC8008000"/>
+<mfgpreviewcolor name="silkscreencolor" color="0xFFFEFEFE"/>
+<mfgpreviewcolor name="backgroundcolor" color="0xFF282828"/>
+<mfgpreviewcolor name="coppercolor" color="0xFFFFBF00"/>
+<mfgpreviewcolor name="substratecolor" color="0xFF786E46"/>
+</mfgpreviewcolors>
 </board>
 </drawing>
-<compatibility>
-<note version="6.3" minversion="6.2.2" severity="warning">
-Since Version 6.2.2 text objects can contain more than one line,
-which will not be processed correctly with this version.
-</note>
-</compatibility>
 </eagle>
