File: Experimental/ESP32/50x33/MySens-easyESP32b-012.sch (EAGLE design)
At the start: 23 parts, among them U2 RFM69HCW, U3 ESP-WROOM-32

Commit message: ESP32
Other:
- note added: "Core"
- note added: "ESP32 MysX"
- note added: "Power-Supply"
- note added: "Radio 2 alternativ"
- note removed: "???? io5 ???"
- note removed: "ATSHA204 authentication chip optional for MySensors"
- note removed: "Achtung"
- note removed: "Crypto"
- note removed: "Div"
- note removed: "Easy PCB - Rev 9"
- note removed: "LAN"
- note removed: "Neu: Pull Wiederstände nur an einer zentralen Stelle im 19.200 Baud Bus... (Steckvariante: mit Spannungsteiler! = 3 Widerstände; Normalerweise niemals an diesem Modul Widerstände verbauen!) Alt:Terminierung mit Pull-Widerständen. Zwischen A und B 150 Ohm, von A 330 Ohm nach VCC, von B 330 Ohm nach GND. Damit wird er Bus auf HIGH gehalten wenn Teilnehmer passiv sind. AC-Widerstand ca. bei 120 Ohm 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"
- note removed: "RFM69(H)W"
- note removed: "RS485"
- note removed: "Radio 1 alternativ"
- note removed: "VDD-Config siehe 1Wire..."
- moved on the sheet: ANT1, ANT2, AP2112, C2, C6, C8, C9, CC0, F2, JP1, MYSX, POWER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
