File: Experimental/ESP32/delete/MySens-easyESP32-012.brd (EAGLE design)
At the start: 33 x 50 mm, 22 parts, among them U2 RFM69HCW, U3 ESP-WROOM-32

Commit message: ESP32 SMD
Parts:
- moved IN-FUSED 0.90 mm to (1.91, 22.9)
- moved TP4056 0.32 mm to (13.3, 13.3), turned to 180 degrees
Routing:
- net IO2: track 56.0 -> 85.9 mm, vias 2 -> 1
- net GND: track 204.8 -> 185.8 mm, vias 3 -> 4
- net IO23: track 59.5 -> 44.7 mm
- net VCC: track 140.5 -> 126.2 mm, vias 3 -> 4
- net IO5: track 29.1 -> 19.9 mm
- net EN: track 60.3 -> 68.8 mm
- net IO17: track 58.8 -> 55.1 mm, vias 2 -> 3
- net IO25: track 39.3 -> 36.4 mm, vias 1 -> 0
- net IO0: track 25.0 -> 22.3 mm
- net UREG: track 66.4 -> 63.8 mm, vias 2 -> 1
- net IN++: track 31.0 -> 28.4 mm, vias 2 -> 0
- net IO14: track 27.7 -> 25.3 mm
- net IO26: track 25.4 -> 23.8 mm
- net IO27: track 38.9 -> 37.7 mm, vias 2 -> 1
- net IO4: track 25.4 -> 26.5 mm, vias 0 -> 1
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