File: Experimental/ESP32/delete/MySens-easyESP32-012.sch (EAGLE design)
At the start: 22 parts, among them U2 RFM69HCW, U3 ESP-WROOM-32

Commit message: ESP32 SMD
Parts:
- removed POWER: (no value), con-lstb:MA04-1
- added IN-FUSED: (no value), pinhead:PINHD-1X1
- TP4056: device tp2112-usw-V2:TP4056-MODULE -> tp2112-usw:TP4056-MODULE
Connections:
- removed net B-: POWER.2, TP4056.B-
- removed net IN+: F2.2, POWER.4
- new net IN-FUSED: F2.2, IN-FUSED.1
- new net N$1: TP4056.B-
- net B+: no longer POWER.1
- net IN-: no longer POWER.3
Changed lines of the file:
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@@
 <part name="GND23" library="SparkFun-Aesthetics" deviceset="GND" device=""/>
 <part name="JP1" library="SparkFun-Jumpers" deviceset="JUMPER-SMT_2_NC_PASTE" device="_NO-SILK"/>
-<part name="TP4056" library="tp2112-usw-V2" deviceset="TP4056-MODULE" device=""/>
+<part name="TP4056" library="tp2112-usw" deviceset="TP4056-MODULE" device=""/>
 <part name="AP2112" library="SparkFun-IC-Power" deviceset="V_REG_AP2112" device="K-3.3V" value="3.3V"/>
 <part name="GND24" library="supply1" deviceset="GND" device=""/>
 <part name="GND5" library="supply1" deviceset="GND" device=""/>
-<part name="POWER" library="con-lstb" deviceset="MA04-1" device=""/>
 <part name="ANT2" library="pinhead" deviceset="PINHD-1X1" device=""/>
 <part name="R7" library="rcl" deviceset="R-EU_" device="M0805" value="100k"/>
+<part name="IN-FUSED" library="pinhead" deviceset="PINHD-1X1" device=""/>
 </parts>
 <sheets>
@@
 <instance part="GND24" gate="1" x="-68.58" y="-160.02"/>
 <instance part="GND5" gate="1" x="-96.52" y="-157.48"/>
-<instance part="POWER" gate="1" x="-93.98" y="-177.8" rot="R90"/>
 <instance part="ANT2" gate="G$1" x="223.52" y="30.48"/>
 <instance part="R7" gate="G$1" x="-55.88" y="-142.24" rot="R180"/>
+<instance part="IN-FUSED" gate="G$1" x="-127" y="-177.8" rot="R270"/>
 </instances>
 <busses>
@@
 <wire x1="-96.52" y1="-144.78" x2="-88.9" y2="-144.78" width="0.1524" layer="91"/>
 <label x="-93.98" y="-147.32" size="1.778" layer="95"/>
-<pinref part="POWER" gate="1" pin="1"/>
 <wire x1="-88.9" y1="-144.78" x2="-88.9" y2="-170.18" width="0.1524" layer="91"/>
 </segment>
@@
 <net name="B-" class="1">
 <segment>
-<pinref part="TP4056" gate="G$1" pin="B-"/>
-<wire x1="-96.52" y1="-149.86" x2="-93.98" y2="-149.86" width="0.1524" layer="91"/>
-<wire x1="-93.98" y1="-149.86" x2="-91.44" y2="-149.86" width="0.1524" layer="91"/>
-<label x="-93.98" y="-149.86" size="1.778" layer="95"/>
-<pinref part="POWER" gate="1" pin="2"/>
 <wire x1="-91.44" y1="-170.18" x2="-91.44" y2="-149.86" width="0.1524" layer="91"/>
 </segment>
@@
 <wire x1="-121.92" y1="-152.4" x2="-121.92" y2="-160.02" width="0.1524" layer="91"/>
 <wire x1="-121.92" y1="-160.02" x2="-121.92" y2="-162.56" width="0.1524" layer="91"/>
-<wire x1="-121.92" y1="-162.56" x2="-93.98" y2="-162.56" width="0.1524" layer="91"/>
-<pinref part="POWER" gate="1" pin="3"/>
-<wire x1="-93.98" y1="-162.56" x2="-93.98" y2="-170.18" width="0.1524" layer="91"/>
-<label x="-109.22" y="-162.56" size="1.778" layer="95"/>
-</segment>
-</net>
-<net name="IN+" class="2">
-<segment>
-<pinref part="POWER" gate="1" pin="4"/>
-<wire x1="-96.52" y1="-170.18" x2="-96.52" y2="-167.64" width="0.1524" layer="91"/>
-<wire x1="-96.52" y1="-167.64" x2="-127" y2="-167.64" width="0.1524" layer="91"/>
-<label x="-109.22" y="-165.1" size="1.778" layer="95"/>
-<pinref part="F2" gate="F1" pin="2"/>
 </segment>
 </net>
@@
 </segment>
 </net>
+<net name="N$1" class="1">
+<segment>
+<pinref part="TP4056" gate="G$1" pin="B-"/>
+<wire x1="-96.52" y1="-149.86" x2="-93.98" y2="-149.86" width="0.1524" layer="91"/>
+<label x="-93.98" y="-149.86" size="1.778" layer="95"/>
+</segment>
+</net>
+<net name="IN-FUSED" class="0">
+<segment>
+<pinref part="F2" gate="F1" pin="2"/>
+<pinref part="IN-FUSED" gate="G$1" pin="1"/>
+<wire x1="-127" y1="-175.26" x2="-127" y2="-167.64" width="0.1524" layer="91"/>
+<label x="-121.92" y="-172.72" size="1.778" layer="95" rot="R270"/>
+</segment>
+</net>
