File: Experimental/ESP32/AddOn/DisplayAddOn_V012.brd (EAGLE design)
At the start: 33 x 50 mm, 7 parts

Commit message: ESP32
Parts:
- removed POWER: (no value), con-lstb:MA04-1
- removed U$1: HELTEC_1.54STANDARD1, display:HELTEC_1.54INCH
- added HELTEK: HELTEC_1.54STANDARD1, display_v2:HELTEC_1.54INCH
- added J1: (no value), SparkFun-Connectors:1X02
- added WAVESHARE: (no value), SparkFun-Connectors:1X08
Connections:
- removed net ???XXX???: U$1.SDI
- removed net B+: POWER.1
- removed net B-: POWER.2
- removed net IN+: POWER.4
- removed net N$2: POWER.3
- new net FREE: J1.1
- net GND: now also HELTEK.GND, WAVESHARE.2; no longer U$1.GND
- net IO13: now also HELTEK.SDI, WAVESHARE.4
- net IO14: now also HELTEK.CLK, WAVESHARE.6; no longer U$1.CLK
- net IO15: now also J1.2, WAVESHARE.8
- net IO26: now also HELTEK.CS, WAVESHARE.5; no longer U$1.CS
- net IO27: now also HELTEK.D/C, WAVESHARE.3; no longer U$1.D/C
- net VCC: now also HELTEK.VCC, WAVESHARE.1; no longer U$1.VCC
Routing:
- net IO13: track 0.00 -> 67.5 mm
- net IO15: track 0.00 -> 37.6 mm
- net IO14: track 24.5 -> 47.7 mm
- net IO26: track 24.5 -> 47.4 mm
- net IO27: track 41.8 -> 56.0 mm
- net GND: track 65.5 -> 77.6 mm, vias 0 -> 26
- net VCC: track 71.0 -> 76.1 mm
- net IO22: track 30.3 -> 32.9 mm
- added copper zone on layer 1, net GND
- added copper zone on layer 16, net GND
Other:
- board text added: "(C) www.neuby.de"
- board text added: "13"
- board text added: "14"
- board text added: "15"
- board text added: "26"
- board text added: "27"
- board text added: "IO15"
- board text added: "IO27"
- board text added: "MysX Display AddOn V0.1"
- board text removed: "5V"
- board text removed: "PluepillGW V01 RS485, RFM69, RFM95"
- board text removed: "SDA"
- board text removed: "SDL"
- board text removed: "UREG"
- board text removed: "easyGW BluePill 0.2 RS485, RFM69, RFM95"
