File: Experimental/ESP32/AddOn/DisplayAddOn_V012.sch (EAGLE design)
At the start: 7 parts

Commit message: ESP32
Parts:
- removed POWER: (no value), con-lstb:MA04-1
- removed U$1: HELTEC_1.54STANDARD1, display:HELTEC_1.54STANDARD1
- added HELTEK: HELTEC_1.54STANDARD1, display_v2:HELTEC_1.54STANDARD1
- added J1: (no value), SparkFun-Connectors:CONN_02
- added WAVESHARE: (no value), SparkFun-Connectors:CONN_08"
Connections:
- removed net ???XXX???: U$1.SDI
- removed net B+: POWER.1
- removed net B-: POWER.2
- removed net IN+: POWER.4
- removed net N$2: POWER.3
- new net FREE: J1.1
- net GND: now also HELTEK.GND, WAVESHARE.2; no longer U$1.GND
- net IO13: now also HELTEK.SDI, WAVESHARE.4
- net IO14: now also HELTEK.CLK, WAVESHARE.6; no longer U$1.CLK
- net IO15: now also J1.2, WAVESHARE.8
- net IO26: now also HELTEK.CS, WAVESHARE.5; no longer U$1.CS
- net IO27: now also HELTEK.D/C, WAVESHARE.3; no longer U$1.D/C
- net VCC: now also HELTEK.VCC, WAVESHARE.1; no longer U$1.VCC
Other:
- note removed: "Kann Weg bei Platzmangel"
- note removed: "Only for mechanical Reasons"
- note removed: "Wenn man die Pins von dem MYSx Stecker: 3.3V, GND, RX, TX, EN und GPIO00 nimmt und einen Standad USB Programmer (z.B. einen FDDI um 1,60€) nimmt und den EN auf RTS und GPIO00 auf DTR verbindet. Dann setzt der Flasher den Chip automatisch in den Flash Mode, führt den Flash durch und macht den Reset und started den geflashten Sketch."
