File: MysX-AddOns/RGBWW-LED/RGBWW-003.brd (EAGLE design)
At the start: 47 x 53 mm, 13 parts, among them Q1 60V/32A/35mΩ, Q2 60V/32A/35mΩ

Commit message: AddOns
Parts:
- removed IRLZ44N-B, IRLZ44N-G, IRLZ44N-R: (no value), PAsystem:TO220AV
- removed U$1: (no value), fhem.logo:LOGO
- added F2: 1812L, ptc-littlefuse:1812L
- added Q3, Q4, Q5: 60V/32A/35mΩ, SparkFun-DiscreteSemi:TO220V
- added RAW1, RAW2: (no value), jumper:SJ
- added SV2: (no value), con-Pinheader:MA11-2
- added U$2: (no value), fhem.logo:LOGO
- added U$3: 2.1MMJACKTHM, adafruit:PJ-102A
- moved R2 51.3 mm to (36.8, 15.2), flipped to the bottom
- moved Q2 47.9 mm to (33.0, 25.4)
- moved Q1 31.6 mm to (33.0, 31.8), turned to 0 degrees
- moved R1 24.6 mm to (36.8, 21.6), turned to 0 degrees
- moved R3 23.0 mm to (31.8, 8.89)
- moved R4 19.1 mm to (36.5, 8.76), turned to 180 degrees
- moved W 4.87 mm to (43.2, 34.3)
- moved R5 4.08 mm to (31.8, 15.2), turned to 0 degrees
- moved RGB 1.79 mm to (43.2, 15.2)
Connections:
- removed net RGB-B: IRLZ44N-B.B, R3.1
- removed net RGB-B-OUT: IRLZ44N-B.C, RGB.4
- removed net RGB-G: IRLZ44N-G.B, R4.1
- removed net RGB-G-OUT: IRLZ44N-G.C, RGB.3
- removed net RGB-R: IRLZ44N-R.B, R5.1
- removed net RGB-R-OUT: IRLZ44N-R.C, RGB.2
- removed net RGB-WW: Q1.1, R1.2
- removed net RGB-WW1: Q2.1, R2.2
- new net A0: Q1.1, R1.2, SV2.8
- new net A1: SV2.14
- new net A2: SV2.16
- new net A3: SV2.15
- new net D10_SS: SV2.20
- new net D11_MOSI: SV2.17
- new net D12_MISO: SV2.18
- new net D13_SCK: SV2.19
- new net D2: SV2.9
- new net D3: Q3.1, R3.2, SV2.10
- new net D5: Q4.1, R4.2, SV2.11
- new net D6: Q5.1, R5.2, SV2.12
- new net D7: SV2.22
- new net D8: Q2.1, R2.2, SV2.13
- new net D9: SV2.21
- new net RESET: SV2.7
- new net RGB-WW-OUT2: Q3.2, RGB.2
- new net RGB-WW-OUT3: Q4.2, RGB.3
- new net RGB-WW-OUT4: Q5.2, RGB.4
- new net RX0: SV2.6
- new net TX1: SV2.5
- new net UREG: RAW2.2, SV2.1
- new net VCC: SV2.2, SV2.3
- new net VIN: F2.P$2, RAW1.1, U$3.TIP
- net +12V: now also F2.P$1, RAW1.2, RAW2.1
- net GND: now also Q3.3, Q4.3, Q5.3, R3.1, R4.1, R5.1, SV2.4, U$3.RING; no longer IRLZ44N-B.E, IRLZ44N-G.E, IRLZ44N-R.E, R3.2, R4.2, R5.2
- net RGB-WW-OUT: now also Q1.2
- net RGB-WW-OUT1: now also Q2.2
Routing:
- net GND: track 0.00 -> 69.2 mm, vias 0 -> 23
- net +12V: track 0.00 -> 49.3 mm, vias 0 -> 2
- net RGB-R: track 37.5 -> 0.00 mm
- net UREG: track 0.00 -> 35.8 mm
- net A0: track 0.00 -> 35.7 mm
- net D3: track 0.00 -> 30.6 mm
- net RGB-B: track 28.0 -> 0.00 mm
- net RGB-G: track 25.2 -> 0.00 mm
- net D5: track 0.00 -> 22.6 mm, vias 0 -> 1
- net D8: track 0.00 -> 22.3 mm
- net RGB-WW-OUT1: track 0.00 -> 16.5 mm
- net RGB-WW-OUT2: track 0.00 -> 15.5 mm
- net RGB-WW-OUT: track 0.00 -> 15.4 mm
- net RGB-WW-OUT3: track 0.00 -> 14.6 mm
- net RGB-WW-OUT4: track 0.00 -> 13.8 mm
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- added copper zone on layer 1, net GND
- removed copper zone on layer 16, net +12V
- removed copper zone on layer 1, net RGB-B-OUT
- removed copper zone on layer 1, net RGB-CW-OUT
- removed copper zone on layer 1, net RGB-G-OUT
- removed copper zone on layer 1, net RGB-R-OUT
- removed copper zone on layer 1, net RGB-WW-OUT
Other:
- board size 47 x 53 mm -> 26 x 47.2 mm
- board text added: "MySX RGBWW0.1"
- board text removed: "3.3V"
- board text removed: "RGBWW1.5"
