File: MySensors-HM-easy-PCB-RFM-CC1101-RS485-NRF/2_Mini/V03/MinieasySens-RFM_V03-Build004.sch (EAGLE design)
At the start: 33 parts, among them IC1 ATSHA204A, IC2 REG1117, IC3 LD117ADT50TR, IC4 LM1117MPX-ADJ, M1 ARDUINO-PRO-MINI-3.3V#NP, U1 RFM69HCW

Commit message: Mini RFM-V03
Parts:
- removed DTR: (no value), pinhead:PINHD-1X1
- removed FTDI: (no value), con-lstb:MA06-1
- removed I2C-2, STEPDWN1, V2-: (no value), pinhead-2:PINHD-1X04_2.54-S
- added ANT2: (no value), pinhead:PINHD-1X1
Connections:
- removed net CTS: FTDI.5
- removed net DTR: DTR.1, FTDI.1
- removed net TX0: FTDI.2
- net A4: no longer I2C-2.3
- net A5: no longer I2C-2.4
- net ANT: now also ANT2.1
- net D4: no longer V2-.3
- net D8: no longer V2-.4
- net GND: no longer FTDI.6, I2C-2.2, STEPDWN1.2, V2-.2
- net RX0: no longer FTDI.3
- net UREG: no longer STEPDWN1.3
- net V2: no longer V2-.1
- net VCC: no longer FTDI.4, I2C-2.1, STEPDWN1.1, STEPDWN1.4
