File: MySensors-HM-easy-PCB-RFM-CC1101-RS485-NRF/2_Mini/V03/MinieasySens-RFM_V03-Build007.brd (EAGLE design)
At the start: 63 x 33 mm, 29 parts, among them IC1 ATSHA204A, IC2 REG1117, IC3 LD117ADT50TR, IC4 LM1117MPX-ADJ, M1 ARDUINO-PRO-MINI-3.3V#NP, U1 RFM69HCW

Commit message: V03
Parts:
- added IC5: AT25DF512C-SSHN-B, microchip:SO-08
- added JP3: JUMPER-SMT_2_NC_TRACE_SILK, SparkFun-Jumpers:SMT-JUMPER_2_NC_TRACE_SILK
- added R5: 56k, resistor:M0805
- moved C1 27.9 mm to (43.2, 16.5), flipped to the top, turned to 270 degrees
- moved R1 11.8 mm to (38.7, 26.0), flipped to the top, turned to 90 degrees
- moved C4 10.9 mm to (34.9, 17.1)
- moved C6 8.84 mm to (18.4, 3.17), turned to 180 degrees
- moved IC1 4.26 mm to (36.2, 9.53)
Connections:
- new net VCC1: IC5.3, IC5.7, IC5.8, JP3.1, R5.2
- net D11_MOSI: now also IC5.5
- net D12_MISO: now also IC5.2
- net D13_SCK: now also IC5.6
- net D4: now also IC5.1, R5.1
- net GND: now also IC5.4
- net VCC: now also JP3.2
Routing:
- net VCC1: track 0.00 -> 37.8 mm
- net D12_MISO: track 72.7 -> 93.2 mm
- net D4: track 0.00 -> 18.0 mm, vias 0 -> 3
- net V2: track 49.7 -> 33.1 mm
- net D10_SS: track 98.8 -> 84.7 mm
- net UREG: track 116.6 -> 103.8 mm
- net A1: track 43.0 -> 31.8 mm, vias 0 -> 1
- net D3: track 24.5 -> 34.4 mm
- net A0: track 28.4 -> 38.0 mm
- net GND: track 223.7 -> 232.7 mm, vias 2 -> 19
- net A5: track 73.6 -> 65.9 mm, vias 3 -> 1
- net D11_MOSI: track 67.6 -> 74.5 mm, vias 1 -> 2
- net A3: track 35.6 -> 28.8 mm
- net VCC: track 150.4 -> 157.0 mm, vias 0 -> 1
- net A4: track 73.2 -> 66.7 mm
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- added copper zone on layer 1, net GND
- added copper zone on layer 16, net GND
Other:
- board text added: "AT25DF512C"
- board text added: "R5"
