File: MySensors-HM-easy-PCB-RFM-CC1101-RS485-NRF/2_Mini/V03/MinieasySens-RFM_V03-Build007.sch (EAGLE design)
At the start: 29 parts, among them IC1 ATSHA204A, IC2 REG1117, IC3 LD117ADT50TR, IC4 LM1117MPX-ADJ, M1 ARDUINO-PRO-MINI-3.3V#NP, U1 RFM69HCW

Commit message: V03
Parts:
- added IC5: AT25DF512C-SSHN-B, microchip:25AA080SN
- added JP3: JUMPER-SMT_2_NC_TRACE_SILK, SparkFun-Jumpers:JUMPER-SMT_2_NC_TRACE_SILK
- added R5: 56k, resistor:R-EU_M0805
Connections:
- new net VCC1: IC5.!HOLD, IC5.!WP, IC5.VCC, JP3.1, R5.2
- net D11_MOSI: now also IC5.SI
- net D12_MISO: now also IC5.SO
- net D13_SCK: now also IC5.SCK
- net D4: now also IC5.!CS, R5.1
- net GND: now also IC5.GND
- net VCC: now also JP3.2
Changed lines of the file:
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@@
 <part name="U1" library="doug" deviceset="RFM69H" device="CW"/>
 <part name="ANT2" library="pinhead" deviceset="PINHD-1X1" device=""/>
+<part name="IC5" library="microchip" deviceset="25*" device="SN" technology="AA080" value="AT25DF512C-SSHN-B"/>
+<part name="GND2" library="supply1" deviceset="GND" device=""/>
+<part name="R5" library="resistor" deviceset="R-EU_" device="M0805" value="56k"/>
+<part name="JP3" library="SparkFun-Jumpers" deviceset="JUMPER-SMT_2_NC_TRACE" device="_SILK"/>
 </parts>
 <sheets>
@@
 <attribute name="VALUE" x="87.63" y="99.06" size="1.778" layer="96"/>
 </instance>
+<instance part="IC5" gate="G$1" x="124.968" y="53.594" smashed="yes">
+<attribute name="NAME" x="114.808" y="64.924" size="1.778" layer="95"/>
+<attribute name="VALUE" x="114.808" y="43.334" size="1.778" layer="96"/>
+</instance>
+<instance part="GND2" gate="1" x="132.588" y="38.354" smashed="yes">
+<attribute name="VALUE" x="130.048" y="35.814" size="1.778" layer="96"/>
+</instance>
+<instance part="R5" gate="G$1" x="102.108" y="61.214" smashed="yes" rot="R90">
+<attribute name="NAME" x="100.6094" y="57.404" size="1.778" layer="95" rot="R90"/>
+<attribute name="VALUE" x="105.41" y="57.404" size="1.778" layer="96" rot="R90"/>
+</instance>
+<instance part="JP3" gate="G$1" x="137.668" y="66.294" smashed="yes">
+<attribute name="NAME" x="135.128" y="68.834" size="1.778" layer="95" font="vector"/>
+<attribute name="VALUE" x="135.128" y="63.754" size="1.778" layer="96" font="vector" align="top-left"/>
+</instance>
 </instances>
 <busses>
@@
 <wire x1="-58.42" y1="96.52" x2="-58.42" y2="83.82" width="0.1524" layer="91"/>
 <label x="-58.42" y="83.82" size="1.778" layer="95" rot="R270" xref="yes"/>
+</segment>
+<segment>
+<pinref part="GND2" gate="1" pin="GND"/>
+<pinref part="IC5" gate="G$1" pin="GND"/>
+<wire x1="132.588" y1="40.894" x2="132.588" y2="43.434" width="0.1524" layer="91"/>
 </segment>
 </net>
@@
 <label x="-63.5" y="83.82" size="1.778" layer="95" rot="R270" xref="yes"/>
 </segment>
+<segment>
+<pinref part="JP3" gate="G$1" pin="2"/>
+<wire x1="142.748" y1="66.294" x2="145.288" y2="66.294" width="0.1524" layer="91"/>
+<label x="145.288" y="66.294" size="1.778" layer="95" xref="yes"/>
+</segment>
 </net>
 <net name="A4" class="0">
@@
 <label x="12.7" y="12.7" size="1.778" layer="95" rot="R270" xref="yes"/>
 </segment>
+<segment>
+<pinref part="IC5" gate="G$1" pin="!CS"/>
+<wire x1="112.268" y1="56.134" x2="102.108" y2="56.134" width="0.1524" layer="91"/>
+<label x="99.568" y="56.134" size="1.778" layer="95" rot="R180" xref="yes"/>
+<pinref part="R5" gate="G$1" pin="1"/>
+<wire x1="102.108" y1="56.134" x2="99.568" y2="56.134" width="0.1524" layer="91"/>
+<junction x="102.108" y="56.134"/>
+</segment>
 </net>
 <net name="D3" class="0">
@@
 <label x="73.66" y="190.5" size="1.778" layer="95"/>
 </segment>
+<segment>
+<pinref part="IC5" gate="G$1" pin="SI"/>
+<wire x1="112.268" y1="53.594" x2="107.188" y2="53.594" width="0.1524" layer="91"/>
+<label x="107.188" y="53.594" size="1.778" layer="95" rot="R180" xref="yes"/>
+</segment>
 </net>
 <net name="D12_MISO" class="0">
@@
 <label x="73.66" y="185.42" size="1.778" layer="95"/>
 </segment>
+<segment>
+<pinref part="IC5" gate="G$1" pin="SO"/>
+<wire x1="140.208" y1="53.594" x2="142.748" y2="53.594" width="0.1524" layer="91"/>
+<label x="142.748" y="53.594" size="1.778" layer="95" xref="yes"/>
+</segment>
 </net>
 <net name="D13_SCK" class="0">
@@
 <wire x1="71.12" y1="180.34" x2="88.9" y2="180.34" width="0.1524" layer="91"/>
 <label x="73.66" y="180.34" size="1.778" layer="95"/>
+</segment>
+<segment>
+<pinref part="IC5" gate="G$1" pin="SCK"/>
+<wire x1="112.268" y1="51.054" x2="99.568" y2="51.054" width="0.1524" layer="91"/>
+<label x="99.568" y="51.054" size="1.778" layer="95" rot="R180" xref="yes"/>
 </segment>
 </net>
@@
 </segment>
 </net>
+<net name="VCC1" class="1">
+<segment>
+<pinref part="IC5" gate="G$1" pin="!HOLD"/>
+<wire x1="112.268" y1="48.514" x2="109.728" y2="48.514" width="0.1524" layer="91"/>
+<wire x1="109.728" y1="48.514" x2="109.728" y2="61.214" width="0.1524" layer="91"/>
+<pinref part="IC5" gate="G$1" pin="!WP"/>
+<wire x1="109.728" y1="61.214" x2="112.268" y2="61.214" width="0.1524" layer="91"/>
+<pinref part="IC5" gate="G$1" pin="VCC"/>
+<wire x1="132.588" y1="66.294" x2="109.728" y2="66.294" width="0.1524" layer="91"/>
+<wire x1="109.728" y1="66.294" x2="109.728" y2="61.214" width="0.1524" layer="91"/>
+<junction x="109.728" y="61.214"/>
+<junction x="109.728" y="66.294"/>
+<wire x1="102.108" y1="66.294" x2="109.728" y2="66.294" width="0.1524" layer="91"/>
+<pinref part="R5" gate="G$1" pin="2"/>
+<pinref part="JP3" gate="G$1" pin="1"/>
+<junction x="132.588" y="66.294"/>
+</segment>
+</net>

Commit message: Schematic
Other:
- note added: "Flash & Crypto optional"
Changed lines of the file:
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@@
 <wire x1="-2.54" y1="73.66" x2="12.065" y2="73.66" width="0.1524" layer="97"/>
 <wire x1="-2.54" y1="73.66" x2="161.925" y2="73.66" width="0.1524" layer="97"/>
-<text x="-93.98" y="58.42" size="1.778" layer="97" rot="R90">Regulator</text>
 <text x="22.86" y="157.48" size="1.778" layer="97">Free Pins</text>
 <text x="45.72" y="205.74" size="1.778" layer="91">RFM69(H)W</text>
 <text x="40.64" y="157.48" size="1.778" layer="97">Nur mit 3,3V Arduino!</text>
 <text x="15.24" y="210.82" size="1.778" layer="97">Radios (nur eins erlaubt!)</text>
+<text x="73.66" y="68.58" size="1.778" layer="97">Flash &amp; Crypto optional</text>
 </plain>
 <instances>
@@
 </segment>
 <segment>
-<wire x1="116.84" y1="203.2" x2="116.84" y2="195.58" width="0.1524" layer="91"/>
-<label x="116.84" y="195.58" size="1.778" layer="95" rot="R270" xref="yes"/>
-</segment>
-<segment>
 <pinref part="C4" gate="G$1" pin="2"/>
 <wire x1="-50.8" y1="50.8" x2="-50.8" y2="45.72" width="0.1524" layer="91"/>
@@
 </segment>
 <segment>
-<wire x1="10.16" y1="20.32" x2="10.16" y2="10.16" width="0.1524" layer="91"/>
-<label x="10.16" y="10.16" size="1.778" layer="95" rot="R270" xref="yes"/>
-</segment>
-<segment>
 <pinref part="IC3" gate="G$1" pin="ADJ"/>
 <pinref part="GND1" gate="1" pin="GND"/>
 <wire x1="-33.02" y1="38.1" x2="-33.02" y2="43.18" width="0.1524" layer="91"/>
-</segment>
-<segment>
-<wire x1="-104.14" y1="63.5" x2="-104.14" y2="55.88" width="0.1524" layer="91"/>
-<label x="-104.14" y="55.88" size="1.778" layer="95" rot="R270" xref="yes"/>
 </segment>
 <segment>
@@
 <junction x="76.2" y="111.76"/>
 <pinref part="U1" gate="G$1" pin="GND_3"/>
-</segment>
-<segment>
-<wire x1="-58.42" y1="96.52" x2="-58.42" y2="83.82" width="0.1524" layer="91"/>
-<label x="-58.42" y="83.82" size="1.778" layer="95" rot="R270" xref="yes"/>
 </segment>
 <segment>
@@
 <label x="25.4" y="48.26" size="1.778" layer="95" rot="R270" xref="yes"/>
 </segment>
-<segment>
-<wire x1="-101.6" y1="63.5" x2="-101.6" y2="49.53" width="0.1524" layer="91"/>
-<label x="-101.6" y="49.53" size="1.778" layer="95" rot="R270" xref="yes"/>
-</segment>
 </net>
 <net name="VCC" class="1">
@@
 <wire x1="-33.02" y1="96.52" x2="-33.02" y2="82.55" width="0.1524" layer="91"/>
 <label x="-33.02" y="82.55" size="1.778" layer="95" rot="R270" xref="yes"/>
-</segment>
-<segment>
-<wire x1="114.3" y1="203.2" x2="114.3" y2="189.23" width="0.1524" layer="91"/>
-<label x="114.3" y="189.23" size="1.778" layer="95" rot="R270" xref="yes"/>
 </segment>
 <segment>
@@
 </segment>
 <segment>
-<wire x1="-106.68" y1="63.5" x2="-106.68" y2="49.53" width="0.1524" layer="91"/>
-<label x="-106.68" y="49.53" size="1.778" layer="95" rot="R270" xref="yes"/>
-</segment>
-<segment>
-<wire x1="-99.06" y1="63.5" x2="-99.06" y2="55.88" width="0.1524" layer="91"/>
-<label x="-99.06" y="55.88" size="1.778" layer="95" rot="R270" xref="yes"/>
-</segment>
-<segment>
 <pinref part="RFM69W" gate="A" pin="VCC"/>
 <wire x1="33.02" y1="165.1" x2="15.24" y2="165.1" width="0.1524" layer="91"/>
@@
 <label x="30.48" y="127" size="1.778" layer="95"/>
 <pinref part="U1" gate="G$1" pin="3.3V"/>
-</segment>
-<segment>
-<wire x1="-63.5" y1="96.52" x2="-63.5" y2="83.82" width="0.1524" layer="91"/>
-<label x="-63.5" y="83.82" size="1.778" layer="95" rot="R270" xref="yes"/>
 </segment>
 <segment>
@@
 </segment>
 <segment>
-<wire x1="119.38" y1="203.2" x2="119.38" y2="189.23" width="0.1524" layer="91"/>
-<label x="119.38" y="189.23" size="1.778" layer="95" rot="R270" xref="yes"/>
-</segment>
-<segment>
 <pinref part="I2C-1" gate="A" pin="4"/>
 <wire x1="-25.4" y1="96.52" x2="-25.4" y2="88.9" width="0.1524" layer="91"/>
@@
 </segment>
 <segment>
-<wire x1="121.92" y1="203.2" x2="121.92" y2="195.58" width="0.1524" layer="91"/>
-<label x="121.92" y="195.58" size="1.778" layer="95" rot="R270" xref="yes"/>
-</segment>
-<segment>
 <pinref part="I2C-1" gate="A" pin="3"/>
 <wire x1="-27.94" y1="96.52" x2="-27.94" y2="82.55" width="0.1524" layer="91"/>
@@
 <wire x1="-7.62" y1="182.88" x2="-2.54" y2="182.88" width="0.1524" layer="91"/>
 <label x="-2.54" y="182.88" size="1.778" layer="95" xref="yes"/>
-</segment>
-<segment>
-<wire x1="12.7" y1="20.32" x2="12.7" y2="12.7" width="0.1524" layer="91"/>
-<label x="12.7" y="12.7" size="1.778" layer="95" rot="R270" xref="yes"/>
 </segment>
 <segment>
@@
 <wire x1="-7.62" y1="193.04" x2="2.54" y2="193.04" width="0.1524" layer="91"/>
 <label x="2.54" y="193.04" size="1.778" layer="95" rot="R90" xref="yes"/>
-</segment>
-<segment>
-<wire x1="15.24" y1="20.32" x2="15.24" y2="12.7" width="0.1524" layer="91"/>
-<label x="15.24" y="10.16" size="1.778" layer="95" rot="R270" xref="yes"/>
 </segment>
 </net>
@@
 <label x="-10.16" y="127" size="1.778" layer="95" rot="R180"/>
 </segment>
-<segment>
-<wire x1="-66.04" y1="96.52" x2="-66.04" y2="91.44" width="0.1524" layer="91"/>
-<label x="-66.04" y="91.44" size="1.778" layer="95" rot="R270" xref="yes"/>
-</segment>
 </net>
 <net name="TX1" class="0">
@@
 <wire x1="-48.26" y1="121.92" x2="-38.1" y2="121.92" width="0.1524" layer="91"/>
 <label x="-48.26" y="121.92" size="1.778" layer="95" rot="R180"/>
-</segment>
-</net>
-<net name="N$2" class="1">
-<segment>
-<wire x1="-20.32" y1="-81.28" x2="-25.4" y2="-81.28" width="0.1524" layer="91"/>
-</segment>
-</net>
-<net name="N$1" class="1">
-<segment>
-<wire x1="-25.4" y1="-91.44" x2="-20.32" y2="-91.44" width="0.1524" layer="91"/>
 </segment>
 </net>
@@
 </segment>
 <segment>
-<wire x1="7.62" y1="12.7" x2="7.62" y2="20.32" width="0.1524" layer="91"/>
-<label x="7.62" y="12.7" size="1.778" layer="95" rot="R270" xref="yes"/>
-</segment>
-<segment>
 <pinref part="V2" gate="G$1" pin="1"/>
 <wire x1="-2.54" y1="20.32" x2="-2.54" y2="12.7" width="0.1524" layer="91"/>
@@
 </segment>
 </net>
-<net name="DTR" class="0">
-<segment>
-<wire x1="-71.12" y1="96.52" x2="-71.12" y2="91.44" width="0.1524" layer="91"/>
-<label x="-71.12" y="91.44" size="1.778" layer="95" rot="R270" xref="yes"/>
-<wire x1="-71.12" y1="96.52" x2="-81.28" y2="96.52" width="0.1524" layer="91"/>
-</segment>
-</net>
-<net name="TX0" class="0">
-<segment>
-<wire x1="-68.58" y1="96.52" x2="-68.58" y2="83.82" width="0.1524" layer="91"/>
-<label x="-68.58" y="83.82" size="1.778" layer="95" rot="R270" xref="yes"/>
-</segment>
-</net>
-<net name="CTS" class="0">
-<segment>
-<wire x1="-60.96" y1="96.52" x2="-60.96" y2="91.44" width="0.1524" layer="91"/>
-<label x="-60.96" y="91.44" size="1.778" layer="95" rot="R270" xref="yes"/>
-</segment>
-</net>
